File: a2402-4069-overdrive.brd (EAGLE design)
At the start: 100 x 80 mm, 42 parts, among them U1 FX2-20P-1.27DS, U2 FX2-20S-1.27DS

Commit message: a2402 routing
Parts:
- removed SA2: 108-0052-EVX, switches:108-0052-EVX
- added C12, C13, C14, C15: 22P, capacitors:C-0805
- added C16: 10U/35V, capacitors-electrolytic:E2-5
- added DA2: NJM2068M, ic-jrc:SO-8
- added O2, O4, O6, O8: 450-AA150(15MM,D,BLACK), hardware:EMPTY
- added O3, O7: 450-CP157(15MM,WHITE/BLACK), hardware:EMPTY
- added O5: 450-CP153(15MM,BLUE/WHITE), hardware:EMPTY
- added O9: 450-CP155(15MM,GRAY/WHITE), hardware:EMPTY
- added R2, R23, R25, R26, R27, R28, R29, R30: 10K, resistors:R-0805
- added R24: 2*B20K(CD), potentiometers:RV11-DUAL
- added R31, R32: 15K, resistors:R-0805
- added R33, R34: 100K, resistors:R-0805
- C1, C2: value 10U/35V -> 330N(FILM); device capacitors-electrolytic:E2-5 -> capacitors:C050-035X075
- C10: value 22P -> 330N(FILM); device capacitors:C-0805 -> capacitors:C050-035X075
- C11: value 100N -> 330N(FILM); device capacitors:C-0805 -> capacitors:C050-035X075
- C3: value 100N -> 10U/35V; device capacitors:C-0805 -> capacitors-electrolytic:E2-5
- C4: value 330N(FILM) -> 10U/35V; device capacitors:C050-035X075 -> capacitors-electrolytic:E2-5
- C5, C6, C7: value 330N(FILM) -> 100N; device capacitors:C050-035X075 -> capacitors:C-0805
- C8: value 22P -> 100N
- R11, R12, R6, R7: value 100K -> 10K
- R14: value 10K -> 2*A1M; device resistors:R-0805 -> potentiometers:RV11-DUAL
- R15: value 10K -> 2*A10K; device resistors:R-0805 -> potentiometers:RV11-DUAL
- R17: value 2*A1M -> 10K; device potentiometers:RV11-DUAL -> resistors:R-0805
- R18: value 2*A10K -> 10K; device potentiometers:RV11-DUAL -> resistors:R-0805
- R4, R9: value 10K -> 100K
- moved C10 267.6 mm to (93.0, 25.0), turned to 90 degrees
- moved R19 254.6 mm to (70.5, 44.5), turned to 180 degrees
- moved R22 249.7 mm to (32.0, 39.0), turned to 180 degrees
- moved DA1 248.4 mm to (70.0, 35.0)
- moved R20 242.7 mm to (32.0, 41.5), turned to 180 degrees
- moved R21 241.3 mm to (32.0, 34.0), turned to 180 degrees
- moved C8 234.5 mm to (33.0, 19.0), turned to 270 degrees
- moved C6 224.3 mm to (73.5, 28.0)
- moved R15 222.3 mm to (83.0, 37.0), turned to 90 degrees
- moved R17 221.2 mm to (74.0, 42.5), turned to 90 degrees
- moved R18 220.7 mm to (69.0, 25.5), turned to 180 degrees
- moved C7 220.2 mm to (33.0, 30.0)
- moved R1 220.1 mm to (17.0, 13.0), turned to 90 degrees
- moved R16 211.7 mm to (73.5, 25.5), turned to 180 degrees
- moved R14 196.6 mm to (83.0, 13.0), turned to 90 degrees
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Connections:
- removed net N$20 (its old number): R1.2', R4.2
- removed net N$25: PCB1.BOUTR', R7.1, SA2.5
- new net N$15: R1.2', R2.2
- new net N$33: R20.2, R24.3', R26.1
- new net N$34: R22.2, R24.3, R29.1
- new net N$35: C15.1, DA2.2, R28.2, R32.1
- new net N$37: C15.2, DA2.1, PCB1.BOUTR', R32.2, R34.1
- new net N$39: DA2.3, R29.2, R30.2
- new net N$40: R23.2, R24.1, R30.1
- new net N$61: DA2.5, R26.2, R27.2
- new net N$64: C14.1, DA2.6, R25.2, R31.1
- new net N$65: R21.2, R24.1', R27.1
- net +15V: now also C3.+, C5.2, C7.2, DA2.8; no longer C1.+, C9.2
- net -15V: now also C4.-, C6.1, C8.1, DA2.4; no longer C11.1, C2.-
- net GND: now also C16.-, C3.-, C4.+, C5.1, C6.2, C7.1, C8.2, R15.1, R15.1', R24.2, R24.2', R25.1, R28.1, R33.2, R34.2; no longer C1.-, C11.2, C2.+, C3.1, R18.1, R18.1', R6.2, R7.2
- net N$1: now also C16.+, C9.2; no longer C3.2
- net N$10: now also R10.2, R12.1; no longer R13.2, R15.1
- net N$11: now also C10.1, R14.2', R14.3'; no longer C6.1, R17.2, R17.3
- net N$12: now also C10.2, R15.3; no longer C6.2, R18.3
- net N$13: now also R15.2, R16.1; no longer R18.2, R19.1
- net N$14: now also C12.1, R16.2, R18.1; no longer C8.1, R19.2, R21.1
- net N$17: now also C12.2, R18.2, R21.1; no longer C8.2, R21.2, SA2.3
- net N$18: now also C2.1, R1.3; no longer C5.1, R1.3'
- net N$19: now also C2.2, R22.1; no longer C5.2, SA2.4
- net N$2: now also R12.2, R14.1'; no longer R15.2, R17.1
- net N$21: now also DD1.13, R3.1, R5.1; no longer DD1.9, R4.1, R8.1
- net N$22: now also DD1.12, R5.2, R7.1; no longer DD1.8, R10.1, R8.2
- net N$23: now also R7.2, R9.1; no longer R10.2, R12.1
- net N$24: now also R11.1, R9.2; no longer R12.2, R14.1
- net N$26: now also DD1.9, R11.2, R13.1; no longer DD1.13, R14.2, R16.1
- net N$27: now also C11.1, DD1.8, R14.2, R14.3; no longer C7.1, DD1.12, R17.2', R17.3'
- net N$28: now also C14.2, DA2.7, R31.2, R33.1; no longer R6.1, SA2.2
- net N$29: now also C11.2, R15.3'; no longer C7.2, R18.3'
- net N$3: now also R13.2, R14.1; no longer R16.2, R17.1'
- net N$30: now also R15.2', R17.1; no longer R18.2', R20.1
- net N$31: now also C13.1, R17.2, R19.1; no longer C10.1, R20.2, R22.1
- net N$32: now also C13.2, R19.2, R23.1; no longer C10.2, R22.2, SA2.6
- net N$4: now also C1.2, R20.1; no longer C4.2, SA2.1
- net N$5: now also C1.1, R1.3'; no longer C4.1, R1.3
- net N$6: now also R2.1, R4.1; no longer R3.1, R5.1
- net N$7: now also R4.2, R6.1; no longer R5.2, R9.1
- net N$8: now also R6.2, R8.1; no longer R11.1, R9.2
- net N$9: now also R10.1, R8.2; no longer R11.2, R13.1
Routing:
- net N$19: track 0.00 -> 75.8 mm, vias 0 -> 1
- net N$4: track 0.00 -> 60.0 mm, vias 0 -> 1
- net -15V: track 0.00 -> 59.2 mm, vias 0 -> 2
- net P+15V: track 0.00 -> 57.1 mm, vias 0 -> 1
- net +15V: track 0.00 -> 53.0 mm, vias 0 -> 2
- net N$16: track 0.00 -> 48.7 mm
- net N$32: track 0.00 -> 48.5 mm
- net N$37: track 0.00 -> 48.3 mm, vias 0 -> 1
- net N$11: track 0.00 -> 45.3 mm
- net N$61: track 0.00 -> 44.8 mm, vias 0 -> 2
- net N$17: track 0.00 -> 43.4 mm
- net N$36: track 0.00 -> 43.3 mm
- net N$28: track 0.00 -> 38.5 mm, vias 0 -> 1
- net N$20: track 0.00 -> 38.2 mm, vias 0 -> 2
- net N$39: track 0.00 -> 31.7 mm, vias 0 -> 2
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- added copper zone on layer 1, net GND
- added copper zone on layer 16, net GND
Other:
- board size 100 x 80 mm -> 100 x 50 mm
