File: a2401-diode-distortion.sch (EAGLE design)
At the start: 39 parts, among them U1 FX2-20P-1.27DS, U2 FX2-20S-1.27DS

Commit message: Replaced bypass switch with blend potentiometer
Parts:
- removed R7: 100K, resistors:100K
- removed SA1, SA2, SA3: 108-0052-EVX, switches:108-0052-EVX
- removed VD10, VD7, VD8, VD9: BAV199, diodes:BAV199
- added C13, C14: 100N, capacitors:100N
- added C7, C8: 22P, capacitors:22P
- added DA3: NJM2068M, ic-jrc:NJM2068M
- added R10, R12, R14, R15, R16, R17, R18, R19, R20, R21: 10K, resistors:10K
- added R22, R23: 15K, resistors:15K
- R6: value 100K -> 2B20K(CD); device resistors:100K -> potentiometers:2B20K(CD)
Connections:
- removed net N$21: SA3.2.NO, VD2.A, VD5.C
- removed net N$22: SA1.2.CM, SA3.2.CM, VD10.C, VD9.A
- removed net N$25: PCB1G$5.OUTR, R7.1, SA2.2.CM
- removed net N$28: PCB1G$4.OUTL, R6.1, SA2.1.CM
- new net N$11: C8.1, DA3.2.IN-, R16.2, R23.1
- new net N$13: DA3.1.IN+, R19.2, R20.2
- new net N$15: R12.2, R14.1, R6.2.CCW
- new net N$50: R18.2, R19.1, R6.1.CCW
- new net N$59: R10.2, R15.1, R6.2.CW
- new net N$64: C7.1, DA3.1.IN-, R21.2, R22.1
- new net N$7: C6.2, DA1.2.OUT, R5.2.CW, R5.2.W, R8.2.CW, VD2.C, VD6.A
- new net N$9: C5.2, DA1.1.OUT, R5.1.CW, R5.1.W, R8.1.CW, VD1.C, VD4.A
- net +15V: now also C13.2, DA3*.V+
- net -15V: now also C14.1, DA3*.V-
- net GND: now also C13.1, C14.2, R16.1, R21.1, R6.1.W, R6.2.W; no longer R6.2, R7.2, SA1.1.NO, SA1.2.NO
- net N$10: now also VD2.A, VD5.C; no longer SA1.2.NC
- net N$12: now also DA3.2.IN+, R14.2, R15.2; no longer C5.2, DA1.1.OUT, R5.1.CW, R5.1.W, R8.1.CW, VD1.C, VD4.A, VD7.C, VD7.CMN, VD8.A
- net N$17: now also C3.2, C5.1, DA1.1.IN-, R3.1; no longer SA3.1.NO
- net N$18: now also DA1.1.IN+, PCB1G$2.INL, R17.1; no longer SA1.1.CM, SA3.1.CM, VD7.A, VD8.C
- net N$19: now also C8.2, DA3.2.OUT, PCB1G$5.OUTR, R23.2; no longer C6.2, DA1.2.OUT, R5.2.CW, R5.2.W, R8.2.CW, VD10.A, VD2.C, VD6.A, VD9.C, VD9.CMN
- net N$24: now also R12.1; no longer SA2.2.NO
- net N$27: now also R18.1; no longer SA2.1.NO
- net N$3: now also C7.2, DA3.1.OUT, PCB1G$4.OUTL, R22.2; no longer DA1.1.IN+, PCB1G$2.INL, SA2.1.NC
- net N$5: now also R17.2, R20.1, R6.1.CW; no longer C3.2, C5.1, DA1.1.IN-, R3.1, SA1.1.NC
- net N$6: now also R10.1; no longer SA2.2.NC
Other:
- moved on the sheet: C1, C10, C11, C12, C2, C3, C4, C5, C6, C9, DA1*, DA1.1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

Commit message: a2401 diode distortion board
Parts:
- added O2, O3, O4: 450-AA150(15MM,D,BLACK), hardware:450-AA150(15MM,D,BLACK)
- added O5: 450-CP155(15MM,GRAY/WHITE), hardware:450-CP155(15MM,GRAY/WHITE)
- added O6: 450-CP157(15MM,WHITE/BLACK), hardware:450-CP157(15MM,WHITE/BLACK)
- added O7: 450-CP153(15MM,BLUE/WHITE), hardware:450-CP153(15MM,BLUE/WHITE)
- C10, C11, C12, C13, C14, C9: value 100N -> 100N(TH); device capacitors:100N -> capacitors:100N(TH)
- C5, C6, C7, C8: value 22P -> 22P(TH); device capacitors:22P -> capacitors:22P(TH)
- DA1, DA3: value NJM2068M -> NE5532P; device ic-jrc:NJM2068M -> ic-ti:NE5532P
- DA2: value NJM5532M -> TL072IP; device ic-jrc:NJM5532M -> ic-ti:TL072IP
- L2, L3: value BLM31AJ601SN1L -> BL01RN1A1F1J; device inductors:BLM31AJ601SN1L -> inductors:BL01RN1A1F1J
- R1, R2: value 4K7 -> 4K7(TH); device resistors:4K7 -> resistors:4K7(TH)
- R10, R12, R14, R15, R16, R17, R18, R19, R20, R21: value 10K -> 10K(TH); device resistors:10K -> resistors:10K(TH)
- R22, R23: value 15K -> 15K(TH); device resistors:15K -> resistors:15K(TH)
- R3, R4: value 33K -> 33K(TH); device resistors:33K -> resistors:33K(TH)
Connections:
- net N$23: now also R8.1.W; no longer R8.2.W
- net N$26: now also R8.2.W; no longer R8.1.W
- net N$7: now also R8.1.CW; no longer R8.2.CW
- net N$9: now also R8.2.CW; no longer R8.1.CW
Other:
- moved on the sheet: C1, C10, C11, C12, C13, C14, C2, C3, C4, C5, C6, C7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
