File: m201-stereo-input.brd (EAGLE design)
At the start: 100 x 50 mm, 83 parts, among them U1 FX2-20P-1.27DS, U2 FX2-20S-1.27DS, U3 ERM1-5MM

Commit message: M201 In T/H
Parts:
- removed C20, C21: 100N, capacitors:C-0805
- removed C22, C23: 22P, capacitors:C-0805
- removed DA4: NJM5532M, ic-jrc:SO-8
- removed DA5: LM2903M, ic-fairchild:SO-8
- removed O5, O7: 450-CP156(15MM,BLACK/WHITE), hardware:EMPTY
- removed O6: 450-AA150(15MM,D,BLACK), hardware:EMPTY
- removed R32, R37, R38: 10K, resistors:R-0805
- removed R33, R35: 2*A10K, potentiometers:RV11-DUAL
- removed R34: 2K2, resistors:R-0805
- removed R36: 1K8, resistors:R-0805
- added R3, R4: 100K(TH), resistors:R-0207/10
- added U10: FX2-20S-1.27DS, hardware:EMPTY
- added U11: ERM1-5MM, hardware:EMPTY
- added U4, U8, U9: NUT-M2-SELFLOCK, hardware:EMPTY
- added U5: FX2-20P-1.27DS, hardware:EMPTY
- added U6, U7: SCREW-M2X8, hardware:EMPTY
- C10, C11, C12, C15, C16, C17, C7, C8, C9: value 100N -> 100N(TH); device capacitors:C-0805 -> capacitors:C050-024X044
- C13, C14: value 22P -> 22P(TH); device capacitors:C-0805 -> capacitors:C050-024X044
- C18, C19: value 100N -> 22P(TH); device capacitors:C-0805 -> capacitors:C050-024X044
- DA1, DA2: value NJM2068M -> NJM2068D; device ic-jrc:SO-8 -> ic-jrc:DIP-8
- DA3: value NJM5532M -> LM2903N; device ic-jrc:SO-8 -> ic-fairchild:DIP-8
- L1, L2: value BLM31AJ601SN1L -> BL01RN1A1F1J; device inductors:1206 -> inductors:BL01RN1A
- O1: value (none) -> 450-AA150(15MM,D,BLACK); device text:EMPTY -> hardware:EMPTY
- O2: value 450-AA150(15MM,D,BLACK) -> 450-CP155(15MM,GRAY/WHITE)
- O3: value 450-CP155(15MM,GRAY/WHITE) -> 450-AA150(15MM,D,BLACK)
- O4: value 450-AA150(15MM,D,BLACK) -> 450-CP156(15MM,BLACK/WHITE)
- PCB1: value rev.B -> M201 rev.C
- R1, R10, R2, R9: value 10K -> 10K(TH); device resistors:R-0805 -> resistors:R-0207/10
- R11: value 10K -> 2*B20K(CD); device resistors:R-0805 -> potentiometers:RV11-DUAL
- R12: value 10K -> 10M(TH); device resistors:R-0805 -> resistors:R-0207/10
- R13: value 2*B20K(CD) -> 100K(TH); device potentiometers:RV11-DUAL -> resistors:R-0207/10
- R14: value 10M -> 10M(TH); device resistors:R-0805 -> resistors:R-0207/10
- R15, R5, R6: value 100K -> 100K(TH); device resistors:R-0805 -> resistors:R-0207/10
- R16: value 10M -> 47K(TH); device resistors:R-0805 -> resistors:R-0207/10
- R17: value 100K -> 47K(TH); device resistors:R-0805 -> resistors:R-0207/10
- R18: value 47K -> 9K1(TH); device resistors:R-0805 -> resistors:R-0207/10
- R19: value 47K -> 2*A10K; device resistors:R-0805 -> potentiometers:RV11-DUAL
- R20: value 9K1 -> 9K1(TH); device resistors:R-0805 -> resistors:R-0207/10
- R21: value 9K1 -> 330K(TH); device resistors:R-0805 -> resistors:R-0207/10
- R22, R23: value 9K1 -> 10K(TH); device resistors:R-0805 -> resistors:R-0207/10
- R24: value 330K -> 22K(TH); device resistors:R-0805 -> resistors:R-0207/10
- R25: value 10K -> 4K7(TH); device resistors:R-0805 -> resistors:R-0207/10
- R26: value 10K -> 100R(TH); device resistors:R-0805 -> resistors:R-0207/10
- R27: value 22K -> 33K(TH); device resistors:R-0805 -> resistors:R-0207/10
- R28: value 4K7 -> 33K(TH); device resistors:R-0805 -> resistors:R-0207/10
- R29: value 100R -> 10K(TH); device resistors:R-0805 -> resistors:R-0207/10
- R30: value 33K -> 2K2(TH); device resistors:R-0805 -> resistors:R-0207/10
- R31: value 33K -> 1K8(TH); device resistors:R-0805 -> resistors:R-0207/10
- R7, R8: value 100K -> 10K(TH); device resistors:R-0805 -> resistors:R-0207/10
- U1: value FX2-20P-1.27DS -> SCREW-M2X8
- U2: value FX2-20S-1.27DS -> SCREW-M2X8
- U3: value ERM1-5MM -> NUT-M2-SELFLOCK
- VD1, VD2: value BAS16 -> 1N4148; device diodes:SOT23 -> diodes:DO35-7
- VT1: value BC848 -> BC548; device transistors-npn:SOT23 -> transistors-npn:TO92
- moved U3 250.8 mm to (94.8, -100.5)
- moved O3 240.2 mm to (79.0, -100.5)
- moved O4 235.8 mm to (81.2, -100.5)
- moved O2 232.2 mm to (76.8, -100.5)
- moved O1 229.8 mm to (74.5, -100.5)
- moved U2 178.7 mm to (92.5, -100.5)
- moved U1 177.0 mm to (90.2, -100.5)
- moved R30 82.2 mm to (12.5, 37.0)
- moved R25 76.7 mm to (16.5, 37.0), turned to 90 degrees
- moved R31 70.5 mm to (5.00, 37.0)
- moved C9 66.0 mm to (13.5, 44.0)
- moved R26 61.1 mm to (14.5, 25.0), turned to 90 degrees
- moved C10 58.2 mm to (35.0, 38.0)
- moved R28 58.2 mm to (74.5, 45.0), turned to 180 degrees
- moved R27 52.8 mm to (74.2, 32.5), turned to 180 degrees
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Connections:
- removed net N$18: DA3.6, DA3.7, PCB1.BOUTL'
- removed net N$20: DA4.6, DA4.7, R37.1
- removed net N$21: DA3.1, DA3.2, PCB1.BOUTR'
- removed net N$22: DA4.1, DA4.2, R38.1
- removed net N$23: DA3.5, R35.2
- removed net N$24: DA4.5, R33.2
- removed net N$25: DA3.3, R35.2'
- removed net N$28: DA4.3, R33.2'
- new net N$30: R11.2', R18.1, R19.3
- new net N$32: R11.2, R19.3', R20.1
- net +15V: now also R12.2, R24.2; no longer C15.2, C17.2, DA4.8, DA5.8, R16.2, R27.2
- net -15V: now also VT1.3; no longer C16.1, C18.1, DA4.4, DA5.4, VT1.2
- net GND: now also R11.1, R11.3', R19.1, R19.1', R22.1, R3.1, R30.2, R31.2, R4.1; no longer C15.1, C16.2, C18.2, C21.1, R10.1, R13.3', R17.1, R24.1, R25.1, R29.1, R33.1, R33.1', R34.2, R35.1, R35.1', R36.2, R9.1
- net LMIX: no longer R37.2
- net N$10: now also R4.2; no longer R6.2
- net N$11: now also C19.2, PCB1.BOUTR', R28.2; no longer C23.2, R31.2, R33.3', R35.3'
- net N$12: now also C18.2, PCB1.BOUTL', R27.2; no longer C22.2, R30.2, R33.3, R35.3
- net N$13: now also C18.1, R22.2, R27.1; no longer C22.1, R25.2, R30.1
- net N$14: now also C19.1, R23.2, R28.1; no longer C23.1, R26.2, R31.1
- net N$15: now also C16.1, R10.2, R11.3, R20.2; no longer C20.1, R12.2, R13.3, R22.2
- net N$17: now also C15.2, R12.1, R13.2, R16.1; no longer C19.2, R14.1, R15.2, R18.1
- net N$19: now also C15.1, R11.1', R18.2, R9.2; no longer C19.1, R11.2, R13.1', R20.2
- net N$2: now also R6.2; no longer R8.2
- net N$26: now also R7.2, R9.1; no longer R11.1, R9.2
- net N$27: now also R10.1, R8.2; no longer R10.2, R12.1
- net N$29: now also R16.2, VD1.A; no longer R18.2, VD1.1
- net N$3: now also R19.2; no longer R13.2', R20.1, R21.2
- net N$31: now also C16.2, R14.1, R15.2, R17.1; no longer C20.2, R16.1, R17.2, R19.1
- net N$4: now also R3.2; no longer R5.2
- net N$44: now also R17.2, VD2.A; no longer R19.2, VD2.1
- net N$45: now also C17.2, DA3.3, DA3.5, R21.2, VD1.C, VD2.C; no longer C21.2, DA5.3, DA5.5, R24.2, VD1.2, VD2.2
- net N$46: now also DA3.2, R25.1, R26.2; no longer DA5.2, R28.1, R29.2
- net N$47: now also DA3.6, R24.1, R25.2; no longer DA5.6, R27.1, R28.2
- net N$48: now also DA3.7, R29.2, R30.1; no longer DA5.7, R32.2, R34.1
- net N$49: now also R29.1, VT1.2; no longer R32.1, VT1.1
- net N$51: now also DA3.1, R31.1, VT1.1; no longer DA5.1, R36.1, VT1.3
- net N$8: now also R19.2'; no longer R13.2, R22.1, R23.2
- net N$9: now also R5.2; no longer R7.2
- net RMIX: no longer R38.2
Routing:
- net -15V: track 196.4 -> 129.5 mm, vias 6 -> 2
- net +15V: track 171.7 -> 117.0 mm, vias 5 -> 0
- net N$11: track 57.3 -> 22.5 mm, vias 1 -> 0
- net N$19: track 69.8 -> 102.5 mm, vias 2 -> 0
- net N$32: track 0.00 -> 30.6 mm
- net N$30: track 0.00 -> 28.9 mm
- net LMIX: track 58.4 -> 31.8 mm, vias 0 -> 1
- net N$25: track 25.7 -> 0.00 mm
- net N$28: track 24.3 -> 0.00 mm
- net N$23: track 23.3 -> 0.00 mm
- net N$24: track 21.7 -> 0.00 mm
- net N$18: track 21.5 -> 0.00 mm
- net RMIX: track 51.7 -> 33.4 mm
- net N$21: track 17.0 -> 0.00 mm
- net N$26: track 9.30 -> 24.5 mm
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
Commit message: PCB Update
Parts:
- PCB1: value M201 rev.C -> M202 rev.C
Routing:
- net -15V: track 129.5 -> 128.4 mm
- net +15V: track 117.0 -> 116.0 mm
- net N$19: track 102.5 -> 101.6 mm
