File: m301-stereo-output.sch (EAGLE design)
At the start: 89 parts, among them U1 ERM1-5MM, U4 G3VM-62C1, U5 FX2-20P-1.27DS, U6 FX2-20S-1.27DS, U7 ERM1-5MM

Commit message: M301 Update
Parts:
- removed C26, C27, C28: 100N, capacitors:100N
- removed DA5: LM2903M, ic-fairchild:LM2903M
- removed HL3, HL4: RED/BLUE(2MMX5MM,CC), optoelectronics:RED/BLUE(2MMX5MM,CC)
- removed O3: 450-CP156(15MM,BLACK/WHITE), hardware:450-CP156(15MM,BLACK/WHITE)
- removed R31: 10M, resistors:10M
- removed R32, R33: 100K, resistors:100K
- removed R34, R35: 47K, resistors:47K
- removed R36: 330K, resistors:330K
- removed R37: 22K, resistors:22K
- removed R38: 4K7, resistors:4K7
- removed R39: 100R, resistors:100R
- removed R40: 2K2, resistors:2K2
- removed R41: 10K, resistors:10K
- removed R42: 1K8, resistors:1K8
- removed U7: ERM1-5MM, hardware:ERM1-5MM
- removed VD5, VD8, VD9: BAS16, diodes:BAS16
- removed VT3: BC848, transistors-npn:BC848
- added HL1: RED/BLUE(2MMX5MM,CC), optoelectronics:RED/BLUE(2MMX5MM,CC)
- added R24: 330K(TH), resistors:330K(TH)
- added R25: 22K(TH), resistors:22K(TH)
- added R27: 100R(TH), resistors:100R(TH)
- added R28, R3, R4: 10K(TH), resistors:10K(TH)
- added U2: SCREW-M2X8, hardware:SCREW-M2X8
- added U3: NUT-M2-SELFLOCK, hardware:NUT-M2-SELFLOCK
- added VD3: 1N4148, diodes:1N4148
- added VT1: BC548, transistors-npn:BC548
- C1, C2, C5, C6: value 22P -> 22P(TH); device capacitors:22P -> capacitors:22P(TH)
- C10: value 100N(FILM) -> 100N(TH); device capacitors:100N(FILM) -> capacitors:100N(TH)
- C13: value 100N -> 33U/25V; device capacitors:100N -> capacitors-electrolytic:33U/25V
- C14, C22: value 100N -> 100N(FILM); device capacitors:100N -> capacitors:100N(FILM)
- C15, C16, C23, C24, C25, C7, C8: value 100N -> 100N(TH); device capacitors:100N -> capacitors:100N(TH)
- C17, C18: value 22P -> 100N(TH); device capacitors:22P -> capacitors:100N(TH)
- C19, C20: value 100N -> 22P(TH); device capacitors:100N -> capacitors:22P(TH)
- C21: value 10U/35V -> 100N(FILM); device capacitors-electrolytic:10U/35V -> capacitors:100N(FILM)
- C9: value 33U/25V -> 100N(TH); device capacitors-electrolytic:33U/25V -> capacitors:100N(TH)
- DA1, DA2: value NJM2068M -> NJM2068D; device ic-jrc:NJM2068M -> ic-jrc:NJM2068D
- DA4: value NE555D -> LM2903N; device ic-logic:NE555D -> ic-fairchild:LM2903N
- L1, L2: value BLM31AJ601SN1L -> BL01RN1A1F1J; device inductors:BLM31AJ601SN1L -> inductors:BL01RN1A1F1J
- O1: value (none) -> 450-AA150(15MM,D,BLACK); device text:TITLE -> hardware:450-AA150(15MM,D,BLACK)
- O2: value 450-AA150(15MM,D,BLACK) -> 450-CP156(15MM,BLACK/WHITE); device hardware:450-AA150(15MM,D,BLACK) -> hardware:450-CP156(15MM,BLACK/WHITE)
- PCB1: value rev.B -> M301 rev.C; device module-footprints:ST2-BOARD-50-CHAIN -> module-footprints:ST2-BOARD-50-END
- R1, R11, R2, R5, R6, R7, R9: value 10K -> 10K(TH); device resistors:10K -> resistors:10K(TH)
- R10: value 2A10K -> 10K(TH); device potentiometers:2A10K -> resistors:10K(TH)
- R12, R13: value 100K -> 33K(TH); device resistors:100K -> resistors:33K(TH)
- R14, R15: value 10K -> 10R(TH); device resistors:10K -> resistors:10R(TH)
- R16, R17: value 33K -> 2R(TH); device resistors:33K -> resistors:2R(TH)
- R18: value 10R(1206) -> 10M(TH); device resistors:10R(1206) -> resistors:10M(TH)
- R19: value 10R(1206) -> 100K(TH); device resistors:10R(1206) -> resistors:100K(TH)
- R20: value 2R(1206) -> 10M(TH); device resistors:2R(1206) -> resistors:10M(TH)
- R21: value 2R(1206) -> 100K(TH); device resistors:2R(1206) -> resistors:100K(TH)
- R22: value 10K -> 47K(TH); device resistors:10K -> resistors:47K(TH)
- R23: value 100K -> 47K(TH); device resistors:100K -> resistors:47K(TH)
- R26: value 1K5 -> 4K7(TH); device resistors:1K5 -> resistors:4K7(TH)
- R29: value 3K3 -> 2K2(TH); device resistors:3K3 -> resistors:2K2(TH)
- R30: value 10M -> 1K8(TH); device resistors:10M -> resistors:1K8(TH)
- R8: value 10K -> 2A10K; device resistors:10K -> potentiometers:2A10K
- U1: value ERM1-5MM -> SCREW-M2X8; device hardware:ERM1-5MM -> hardware:SCREW-M2X8
- U4: value G3VM-62C1 -> NUT-M2-SELFLOCK; device optoelectronics:G3VM-62C1 -> hardware:NUT-M2-SELFLOCK
- U5: value FX2-20P-1.27DS -> FX2-20S-1.27DS; device hardware:FX2-20P-1.27DS -> hardware:FX2-20S-1.27DS
- U6: value FX2-20S-1.27DS -> ERM1-5MM; device hardware:FX2-20S-1.27DS -> hardware:ERM1-5MM
- VD1: value BAV199 -> DF01M; device diodes:BAV199 -> diodes:DF01M
- VD2: value BAV199 -> 1N4148; device diodes:BAV199 -> diodes:1N4148
Connections:
- removed net CHAIN+15: PCB1G$10.P+15V, R29.2, U4.1B.S2
- removed net N$2: PCB1G$7.RFBK', R13.2
- removed net N$27: C22.2, DA4.1.CONTROL
- removed net N$28: C21.+, DA4.1.!TRIGGER, DA4.1.THRESHOLD, R23.1, VD5.A
- removed net N$29: R26.2, U4.1A.A
- removed net N$31: DA4.1.OUT, U4.2A.C
- removed net N$36: U4.1A.C, U4.2A.A
- removed net N$4: PCB1G$7.LFBK', R12.2
- removed net N$41: PCB1G$6.CV1, PCB1G$7.CV1'
- removed net N$42: PCB1G$6.CV2, PCB1G$7.CV2'
- removed net N$44: HL3.A2, R29.1
- removed net N$51: PCB1G$10.P-15V, U4.2B.S2
- removed net SENSE: PCB1G$7.SENSE', R22.2, R23.2, R26.1, VD5.C
- net +15V: now also C17.2, C9.2, DA4*.V+, R18.2, R20.2, R25.2; no longer C13.2, C27.2, DA5*.V+, R30.2, R31.2, R37.2, VD2.C
- net -15V: now also C10.1, C18.1, HL1.K, VT1.E; no longer C14.1, C21.-, C22.1, C23.1, C28.1, DA5*.V-, HL3.K, HL4.K, R22.1, VD2.A, VT3.E
- net GND: now also C10.2, C17.1, C18.2, C21.1, C22.1, C25.1, C9.1, R10.1, R11.1, R19.1, R21.1, R24.1, R27.1, R29.2, R30.2, R8.1.CCW, R8.2.CCW; no longer C13.1, C14.2, C19.1, C20.1, C23.2, C26.1, C27.1, C28.2, DA4*.V+, DA4.1.!RESET, R10.1.CCW, R10.2.CCW, R12.1, R13.1, R14.1, R15.1, R32.1, R33.1, R36.1, R39.1, R40.2, R42.2
- net LMIX: now also R9.1; no longer R11.1
- net N$1: no longer U4.1B.S1
- net N$10: now also C13.-, C14.2, C24.1, R8.1.CW; no longer C11.-, C12.2, C25.1, PCB1G$5.OUTR, R10.1.CW
- net N$11: now also C19.2, R12.2, R14.2, VD1.AC1; no longer C17.2, R18.2, R20.2, VD1.CMN
- net N$12: now also C19.1, R10.2, R12.1; no longer C17.1, R14.2, R16.1
- net N$13: now also R22.2, VD2.A; no longer R34.2, VD8.A
- net N$14: now also R14.1; no longer R18.1
- net N$15: now also C11.-, C12.2, C23.1, R8.2.CW; no longer C10.2, C24.1, C9.-, PCB1G$4.OUTL, R10.2.CW
- net N$16: now also C21.2, R16.1; no longer C19.2, R20.1
- net N$17: now also C23.2, R18.1, R19.2, R22.1; no longer C24.2, R30.1, R32.2, R34.1
- net N$18: now also C24.2, R20.1, R21.2, R23.1; no longer C25.2, R31.1, R33.2, R35.1
- net N$20: now also R23.2, VD3.A; no longer R35.2, VD9.A
- net N$21: now also C25.2, DA4.1.IN+, DA4.2.IN+, R24.2, VD2.C, VD3.C; no longer C26.2, DA5.1.IN+, DA5.2.IN+, R36.2, VD8.C, VD9.C
- net N$22: now also C20.1, R11.2, R13.1; no longer C18.1, R15.2, R17.1
- net N$23: now also DA4.1.IN-, R26.1, R27.2; no longer DA5.1.IN-, R38.1, R39.2
- net N$24: now also C20.2, R13.2, R15.2, VD1.AC2; no longer C18.2, R19.2, R21.2, VD2.CMN
- net N$25: now also DA4.1.OUT, HL1.A2, R30.1, VT1.C; no longer DA5.1.OUT, HL4.A2, R42.1, VT3.C
- net N$3: now also R8.1.W; no longer R10.1.W
- net N$39: now also R7.2; no longer R9.2
- net N$40: now also R9.2; no longer R11.2
- net N$45: now also R15.1; no longer R19.1
- net N$46: now also C22.2, R17.1; no longer C20.2, R21.1
- net N$47: now also DA4.2.IN-, R25.1, R26.2; no longer DA5.2.IN-, R37.1, R38.2
- net N$48: now also DA4.2.OUT, HL1.A1, R28.2, R29.1; no longer DA5.2.OUT, HL4.A1, R40.1, R41.2
- net N$49: now also R28.1, VT1.B; no longer R41.1, VT3.B
- net N$5: no longer U4.2B.S1
- net N$54: now also R3.2, R5.1; no longer R5.2, R7.1
- net N$55: now also C11.+, C12.1, R5.2; no longer C10.1, C9.+, R7.2
- net N$56: now also R4.2, R6.1; no longer R6.2, R8.1
- net N$57: now also C13.+, C14.1, R6.2; no longer C11.+, C12.1, R8.2
- net N$7: now also R3.1; no longer R5.1
- net N$8: now also R4.1; no longer R6.1
- net N$9: now also R8.2.W; no longer R10.2.W
- net RMIX: now also R7.1; no longer R9.1
Other:
- moved on the sheet: C1, C10, C11, C12, C14, C15, C16, C17, C18, C19, C2, C20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

Commit message: PCB Update
Parts:
- PCB1: value M301 rev.C -> M303 rev.C
Changed lines of the file:
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@@
 <part name="C9" library="capacitors" deviceset="?" device="100N(TH)" value="100N(TH)"/>
 <part name="C10" library="capacitors" deviceset="?" device="100N(TH)" value="100N(TH)"/>
-<part name="PCB1" library="module-footprints" deviceset="ST2-BOARD-50-END" device="" value="M301 rev.C"/>
+<part name="PCB1" library="module-footprints" deviceset="ST2-BOARD-50-END" device="" value="M303 rev.C"/>
 <part name="U1" library="hardware" deviceset="*?" device="SCREW-M2X8"/>
 <part name="U2" library="hardware" deviceset="*?" device="SCREW-M2X8"/>
