File: a201-kill-eq.sch (EAGLE design)
At the start: 86 parts, among them U10 NUT-M2-SELFLOCK, U11 FX2-20S-1.27DS, U2 SCREW-M2X8, U3 SCREW-M2X8, U4 NUT-M2-SELFLOCK, U5 NUT-M2-SELFLOCK, U6 FX2-20P-1.27DS, U7 SCREW-M2X8, U8 SCREW-M2X8, U9 NUT-M2-SELFLOCK

Commit message: PCB Update
Parts:
- PCB1: value A201 rev.A -> A212 rev.A
Changed lines of the file:
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@@
 </classes>
 <parts>
-<part name="PCB1" library="module-footprints" deviceset="ST2-BOARD-?" device="50" value="A201 rev.A"/>
+<part name="PCB1" library="module-footprints" deviceset="ST2-BOARD-?" device="50" value="A212 rev.A"/>
 <part name="U6" library="hardware" deviceset="?" device="FX2-20P-1.27DS"/>
 <part name="U11" library="hardware" deviceset="?" device="FX2-20S-1.27DS"/>
