File: a202-4-band-eq.brd (EAGLE design)
At the start: 100 x 50 mm, 71 parts, among them U1 SCREW-M2X8, U10 FX2-20S-1.27DS, U2 SCREW-M2X8, U3 NUT-M2-SELFLOCK, U4 NUT-M2-SELFLOCK, U5 FX2-20P-1.27DS, U6 SCREW-M2X8, U7 SCREW-M2X8, U8 NUT-M2-SELFLOCK, U9 NUT-M2-SELFLOCK

Commit message: A202 Routing Update
Parts:
- moved R26 2.00 mm to (53.0, 16.0)
- moved R32 2.00 mm to (53.0, 14.0)
Routing:
- net N$17: track 38.0 -> 40.3 mm
- net N$39: track 3.97 -> 5.75 mm
- net N$34: track 46.8 -> 47.7 mm
Changed lines of the file:
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@@
 <attribute name="MOUSER" value="80-PHE426DJ4220JR05" x="184" y="192" size="1.778" layer="27" rot="R180" display="off"/>
 </element>
-<element name="R32" library="resistors" package="R-0207/10" value="27K(TH)" x="53" y="16" rot="R180"/>
-<element name="R26" library="resistors" package="R-0207/10" value="27K(TH)" x="53" y="14"/>
+<element name="R32" library="resistors" package="R-0207/10" value="27K(TH)" x="53" y="14" rot="R180"/>
+<element name="R26" library="resistors" package="R-0207/10" value="27K(TH)" x="53" y="16"/>
 <element name="R31" library="resistors" package="R-0207/10" value="100K(TH)" x="73" y="40" rot="R270">
 <attribute name="MOUSER" value="71-RN55D-F-100K" x="-71" y="119" size="1.778" layer="27" rot="R270" display="off"/>
@@
 <contactref element="C8" pad="2"/>
 <wire x1="63.46" y1="9" x2="57.75" y2="9" width="0.254" layer="1"/>
-<wire x1="57.75" y1="9" x2="51.75" y2="15" width="0.254" layer="1"/>
-<wire x1="51.75" y1="15" x2="34.92" y2="15" width="0.254" layer="1"/>
-<wire x1="34.92" y1="15" x2="30" y2="19.92" width="0.254" layer="1"/>
+<wire x1="57.75" y1="9" x2="49.75" y2="17" width="0.254" layer="1"/>
+<wire x1="35.17" y1="14.75" x2="30" y2="19.92" width="0.254" layer="1"/>
+<wire x1="49.75" y1="17" x2="47.5" y2="17" width="0.254" layer="1"/>
+<wire x1="47.5" y1="17" x2="46.75" y2="16.25" width="0.254" layer="1"/>
+<wire x1="46.75" y1="16.25" x2="46.75" y2="15.5" width="0.254" layer="1"/>
+<wire x1="46.75" y1="15.5" x2="46" y2="14.75" width="0.254" layer="1"/>
+<wire x1="46" y1="14.75" x2="35.17" y2="14.75" width="0.254" layer="1"/>
 </signal>
 <signal name="N$18">
@@
 <wire x1="63.46" y1="11.96" x2="61.25" y2="9.75" width="0.254" layer="1"/>
 <wire x1="61.25" y1="9.75" x2="58" y2="9.75" width="0.254" layer="1"/>
-<wire x1="58" y1="9.75" x2="50.75" y2="17" width="0.254" layer="1"/>
-<wire x1="50.75" y1="17" x2="47.25" y2="17" width="0.254" layer="1"/>
-<wire x1="47.25" y1="17" x2="45.75" y2="15.5" width="0.254" layer="1"/>
-<wire x1="45.75" y1="15.5" x2="38.25" y2="15.5" width="0.254" layer="1"/>
+<wire x1="45.5" y1="15.5" x2="38.25" y2="15.5" width="0.254" layer="1"/>
 <wire x1="38.25" y1="15.5" x2="36.25" y2="17.5" width="0.254" layer="1"/>
 <via x="36.25" y="17.5" extent="1-16" drill="0.5"/>
 <wire x1="36.25" y1="17.5" x2="36.25" y2="31.67" width="0.254" layer="16"/>
+<wire x1="45.5" y1="15.5" x2="46" y2="16" width="0.254" layer="1"/>
+<wire x1="46" y1="16" x2="46" y2="16.5" width="0.254" layer="1"/>
+<wire x1="46" y1="16.5" x2="47.25" y2="17.75" width="0.254" layer="1"/>
+<wire x1="47.25" y1="17.75" x2="50" y2="17.75" width="0.254" layer="1"/>
+<wire x1="50" y1="17.75" x2="58" y2="9.75" width="0.254" layer="1"/>
 </signal>
 <signal name="N$35">
@@
 <wire x1="75.19" y1="43.81" x2="71.35" y2="43.81" width="0.254" layer="16"/>
 <wire x1="71.35" y1="43.81" x2="68.54" y2="41" width="0.254" layer="16"/>
-<wire x1="58.08" y1="16" x2="58.08" y2="29.83" width="0.254" layer="16"/>
 <via x="58.08" y="29.83" extent="1-16" drill="0.5"/>
 <wire x1="61.25" y1="36" x2="66.75" y2="36" width="0.254" layer="1"/>
@@
 <wire x1="58.75" y1="30.5" x2="58.75" y2="33.5" width="0.254" layer="1"/>
 <wire x1="58.75" y1="33.5" x2="61.25" y2="36" width="0.254" layer="1"/>
+<wire x1="58.08" y1="29.83" x2="58.08" y2="16" width="0.254" layer="16"/>
 <wire x1="58.08" y1="14" x2="58.08" y2="16" width="0.254" layer="16"/>
 </signal>
@@
 <contactref element="R26" pad="1"/>
 <contactref element="C18" pad="2"/>
-<wire x1="47.92" y1="14" x2="47.54" y2="14" width="0.254" layer="1"/>
-<wire x1="47.54" y1="14" x2="45" y2="11.46" width="0.254" layer="1"/>
+<wire x1="47.92" y1="16" x2="47.92" y2="15.67" width="0.254" layer="1"/>
+<wire x1="47.92" y1="15.67" x2="45" y2="12.75" width="0.254" layer="1"/>
+<wire x1="45" y1="12.75" x2="45" y2="11.46" width="0.254" layer="1"/>
 </signal>
 <signal name="N$40">

Commit message: Add Potentiometer Knobs
Parts:
- added O1, O2, O3, O4: 450-AA150(15MM,D,BLACK), hardware:EMPTY
- added O5, O6, O7, O8: 450-CP153(15MM,BLUE/WHITE), hardware:EMPTY
Changed lines of the file:
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@@
 <attribute name="MOUSER" value="81-RCER71H104K0A2H3B" x="12" y="-171" size="1.778" layer="27" display="off"/>
+</element>
+<element name="O1" library="hardware" package="EMPTY" value="450-AA150(15MM,D,BLACK)" x="-8" y="-109.25">
+<attribute name="MOUSER" value="450-AA150" x="-8" y="-109.25" size="1.778" layer="27" display="off"/>
+</element>
+<element name="O2" library="hardware" package="EMPTY" value="450-AA150(15MM,D,BLACK)" x="-9" y="-110.5">
+<attribute name="MOUSER" value="450-AA150" x="-9" y="-110.5" size="1.778" layer="27" display="off"/>
+</element>
+<element name="O3" library="hardware" package="EMPTY" value="450-AA150(15MM,D,BLACK)" x="-10" y="-111.75">
+<attribute name="MOUSER" value="450-AA150" x="-10" y="-111.75" size="1.778" layer="27" display="off"/>
+</element>
+<element name="O4" library="hardware" package="EMPTY" value="450-AA150(15MM,D,BLACK)" x="-11" y="-113">
+<attribute name="MOUSER" value="450-AA150" x="-11" y="-113" size="1.778" layer="27" display="off"/>
+</element>
+<element name="O5" library="hardware" package="EMPTY" value="450-CP153(15MM,BLUE/WHITE)" x="-12" y="-114.25">
+<attribute name="MOUSER" value="450-CP153" x="-12" y="-114.25" size="1.778" layer="27" display="off"/>
+</element>
+<element name="O6" library="hardware" package="EMPTY" value="450-CP153(15MM,BLUE/WHITE)" x="-13" y="-115.5">
+<attribute name="MOUSER" value="450-CP153" x="-13" y="-115.5" size="1.778" layer="27" display="off"/>
+</element>
+<element name="O7" library="hardware" package="EMPTY" value="450-CP153(15MM,BLUE/WHITE)" x="-14" y="-116.75">
+<attribute name="MOUSER" value="450-CP153" x="-14" y="-116.75" size="1.778" layer="27" display="off"/>
+</element>
+<element name="O8" library="hardware" package="EMPTY" value="450-CP153(15MM,BLUE/WHITE)" x="-15" y="-118">
+<attribute name="MOUSER" value="450-CP153" x="-15" y="-118" size="1.778" layer="27" display="off"/>
 </element>
 </elements>

Commit message: PCB Update
Parts:
- PCB1: value A202 rev.A -> A210 rev.A
Routing:
- net N$7: track 51.0 -> 49.7 mm
- net N$37: track 68.6 -> 67.7 mm
- net N$47: track 109.0 -> 108.2 mm
- net N$14: track 129.3 -> 128.5 mm
- net N$45: track 104.0 -> 103.2 mm
- net N$23: track 17.6 -> 17.0 mm
- net N$32: track 124.8 -> 124.2 mm
- net N$29: track 109.9 -> 109.4 mm
- net N$24: track 26.0 -> 25.5 mm
- net N$27: track 73.1 -> 72.6 mm
- net N$36: track 50.0 -> 49.5 mm
