File: a202-4-band-eq.sch (EAGLE design)
At the start: 71 parts, among them U1 SCREW-M2X8, U10 FX2-20S-1.27DS, U2 SCREW-M2X8, U3 NUT-M2-SELFLOCK, U4 NUT-M2-SELFLOCK, U5 FX2-20P-1.27DS, U6 SCREW-M2X8, U7 SCREW-M2X8, U8 NUT-M2-SELFLOCK, U9 NUT-M2-SELFLOCK

Commit message: Add Potentiometer Knobs
Parts:
- added O1, O2, O3, O4: 450-AA150(15MM,D,BLACK), hardware:450-AA150(15MM,D,BLACK)
- added O5, O6, O7, O8: 450-CP153(15MM,BLUE/WHITE), hardware:450-CP153(15MM,BLUE/WHITE)
Changed lines of the file:
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@@
 <part name="C6" library="capacitors" deviceset="?" device="100N(TH)"/>
 <part name="GND1" library="supply" deviceset="GND" device=""/>
+<part name="O1" library="hardware" deviceset="450-AA?" device="150(15MM,D,BLACK)"/>
+<part name="O2" library="hardware" deviceset="450-AA?" device="150(15MM,D,BLACK)"/>
+<part name="O3" library="hardware" deviceset="450-AA?" device="150(15MM,D,BLACK)"/>
+<part name="O4" library="hardware" deviceset="450-AA?" device="150(15MM,D,BLACK)"/>
+<part name="O5" library="hardware" deviceset="450-C?" device="P153(15MM,BLUE/WHITE)"/>
+<part name="O6" library="hardware" deviceset="450-C?" device="P153(15MM,BLUE/WHITE)"/>
+<part name="O7" library="hardware" deviceset="450-C?" device="P153(15MM,BLUE/WHITE)"/>
+<part name="O8" library="hardware" deviceset="450-C?" device="P153(15MM,BLUE/WHITE)"/>
 </parts>
 <sheets>
@@
 <instance part="DA1" gate="*" x="78.74" y="-76.2"/>
 <instance part="DA2" gate="*" x="93.98" y="-76.2"/>
+<instance part="O1" gate="G$1" x="58.42" y="-106.68"/>
+<instance part="O2" gate="G$1" x="58.42" y="-124.46"/>
+<instance part="O3" gate="G$1" x="58.42" y="-142.24"/>
+<instance part="O4" gate="G$1" x="58.42" y="-160.02"/>
+<instance part="O5" gate="G$1" x="58.42" y="-106.68"/>
+<instance part="O6" gate="G$1" x="58.42" y="-124.46"/>
+<instance part="O7" gate="G$1" x="58.42" y="-142.24"/>
+<instance part="O8" gate="G$1" x="58.42" y="-160.02"/>
 </instances>
 <busses>

Commit message: PCB Update
Parts:
- PCB1: value A202 rev.A -> A210 rev.A
Changed lines of the file:
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@@
 </classes>
 <parts>
-<part name="PCB1" library="module-footprints" deviceset="ST2-BOARD-?" device="50" value="A202 rev.A"/>
+<part name="PCB1" library="module-footprints" deviceset="ST2-BOARD-?" device="50" value="A210 rev.A"/>
 <part name="U5" library="hardware" deviceset="?" device="FX2-20P-1.27DS"/>
 <part name="U10" library="hardware" deviceset="?" device="FX2-20S-1.27DS"/>
