File: a402-4069-overdrive.brd (EAGLE design)
At the start: 100 x 50 mm, 68 parts, among them U1 FX2-20P-1.27DS, U2 FX2-20S-1.27DS

Commit message: PCB Update
Parts:
- removed O1: (no value), text:EMPTY
- added U10, U7, U8, U9: NUT-M2-SELFLOCK, hardware:EMPTY
- added U3, U4, U5, U6: SCREW-M2X8, hardware:EMPTY
- PCB1: value rev.A -> A406 rev.A
Changed lines of the file:
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@@
 <?xml version="1.0" encoding="utf-8"?>
 <!DOCTYPE eagle SYSTEM "eagle.dtd">
-<eagle version="7.5.0">
+<eagle version="7.5.1">
 <drawing>
 <settings>
@@
 </autorouter>
 <elements>
-<element name="O1" library="text" package="EMPTY" value="" x="41" y="-96"/>
-<element name="PCB1" library="module-footprints" package="ST2-BOARD-50" value="rev.A" x="0" y="0"/>
+<element name="PCB1" library="module-footprints" package="ST2-BOARD-50" value="A406 rev.A" x="0" y="0"/>
 <element name="U1" library="hardware" package="EMPTY" value="FX2-20P-1.27DS" x="44" y="-96">
 <attribute name="MOUSER" value="798-FX2-20P-1.27DS71" x="-1" y="-63" size="1.778" layer="27" display="off"/>
@@
 <attribute name="MOUSER" value="647-USW1V100MDD" x="43" y="18.5" size="1.778" layer="27" rot="R270" display="off"/>
 </element>
+<element name="U3" library="hardware" package="EMPTY" value="SCREW-M2X8" x="-16" y="-113.25"/>
+<element name="U4" library="hardware" package="EMPTY" value="SCREW-M2X8" x="-17" y="-114.5"/>
+<element name="U5" library="hardware" package="EMPTY" value="SCREW-M2X8" x="-18" y="-115.75"/>
+<element name="U6" library="hardware" package="EMPTY" value="SCREW-M2X8" x="-19" y="-117"/>
+<element name="U7" library="hardware" package="EMPTY" value="NUT-M2-SELFLOCK" x="-20" y="-118.25"/>
+<element name="U8" library="hardware" package="EMPTY" value="NUT-M2-SELFLOCK" x="-21" y="-119.5"/>
+<element name="U9" library="hardware" package="EMPTY" value="NUT-M2-SELFLOCK" x="-22" y="-120.75"/>
+<element name="U10" library="hardware" package="EMPTY" value="NUT-M2-SELFLOCK" x="-23" y="-122"/>
 </elements>
 <signals>
@@
 <contactref element="R15" pad="2"/>
 <contactref element="R16" pad="1"/>
-<wire x1="93.5" y1="29" x2="95.45710625" y2="30.95710625" width="0.254" layer="1"/>
+<wire x1="86.6642125" y1="29" x2="93.0857875" y2="29" width="0.254" layer="1"/>
+<wire x1="93.0857875" y1="29" x2="93.79289375" y2="29.29289375" width="0.254" layer="1" curve="45"/>
+<wire x1="93.79289375" y1="29.29289375" x2="95.45710625" y2="30.95710625" width="0.254" layer="1"/>
 <wire x1="95.45710625" y1="30.95710625" x2="95.75" y2="31.6642125" width="0.254" layer="1" curve="45"/>
 <wire x1="94" y1="38" x2="95.45710625" y2="36.54289375" width="0.254" layer="1"/>
 <wire x1="95.45710625" y1="36.54289375" x2="95.75" y2="35.8357875" width="0.254" layer="1" curve="-45"/>
 <wire x1="95.75" y1="35.8357875" x2="95.75" y2="31.6642125" width="0.254" layer="1"/>
-<wire x1="86.25" y1="29" x2="93.5" y2="29" width="0.254" layer="1"/>
-<wire x1="82.75" y1="25.5" x2="86.25" y2="29" width="0.254" layer="1"/>
-<wire x1="74.75" y1="25.5" x2="82.75" y2="25.5" width="0.254" layer="1"/>
+<wire x1="83.04289375" y1="25.79289375" x2="85.95710625" y2="28.70710625" width="0.254" layer="1"/>
+<wire x1="85.95710625" y1="28.70710625" x2="86.6642125" y2="29" width="0.254" layer="1" curve="-45"/>
+<wire x1="74.75" y1="25.5" x2="82.3357875" y2="25.5" width="0.254" layer="1"/>
+<wire x1="82.3357875" y1="25.5" x2="83.04289375" y2="25.79289375" width="0.254" layer="1" curve="45"/>
 <wire x1="74.5" y1="25.25" x2="74.75" y2="25.5" width="0.254" layer="1"/>
 <wire x1="74.25" y1="25.5" x2="74.5" y2="25.25" width="0.254" layer="1"/>
