File: d701-vs1053-synth.brd (EAGLE design)
At the start: 100 x 50 mm, 88 parts, among them U1 FX2-20P-1.27DS, U2 FX2-20S-1.27DS, U3 ERM1-5MM

Commit message: d701 routing update
Parts:
- removed C37: 22P, capacitors:C-0805
- removed C38: 10U/35V, capacitors-electrolytic:E2-5
- added C11, C12: 1U, capacitors:C-0805
- C10: value 1U -> 10U/35V; device capacitors:C-0805 -> capacitors-electrolytic:E2-5
- C14: value 1U -> 100N
- C15: value 100N -> 47N(FILM); device capacitors:C-0805 -> capacitors:C050-025X075
- C16: value 47N(FILM) -> 100N; device capacitors:C050-025X075 -> capacitors:C-0805
- C18, C22: value 100N -> 10N(FILM); device capacitors:C-0805 -> capacitors:C050-025X075
- C19, C23: value 10N(FILM) -> 100N; device capacitors:C050-025X075 -> capacitors:C-0805
- C25, C27: value 100N -> 3N3(FILM); device capacitors:C-0805 -> capacitors:C050-025X075
- C26, C28: value 3N3(FILM) -> 100N; device capacitors:C050-025X075 -> capacitors:C-0805
- C29: value 100N -> 100N(FILM); device capacitors:C-0805 -> capacitors:C050-025X075
- C3: value 100N -> 10U/35V; device capacitors:C-0805 -> capacitors-electrolytic:E2-5
- C30, C32: value 100N(FILM) -> 33U/25V; device capacitors:C050-025X075 -> capacitors-electrolytic:E2,5-7
- C31: value 47U/35V -> 100N(FILM); device capacitors-electrolytic:E3,5-8 -> capacitors:C050-025X075
- C33: value 47U/35V -> 100N; device capacitors-electrolytic:E3,5-8 -> capacitors:C-0805
- C35: value 100N -> 22P
- C5: value 10U/35V -> 100N; device capacitors-electrolytic:E2-5 -> capacitors:C-0805
- moved C5 48.9 mm to (74.5, 17.0)
- moved C35 46.5 mm to (71.0, 32.0), turned to 180 degrees
- moved C1 36.5 mm to (29.0, 43.0), turned to 270 degrees
- moved C33 34.4 mm to (15.0, 13.5), turned to 0 degrees
- moved C16 32.4 mm to (14.0, 40.0), turned to 270 degrees
- moved C29 30.4 mm to (45.8, 27.8), turned to 90 degrees
- moved C27 29.4 mm to (39.5, 32.0), turned to 180 degrees
- moved C25 27.7 mm to (39.5, 23.0), turned to 180 degrees
- moved C28 25.7 mm to (16.0, 21.5), turned to 270 degrees
- moved C20 24.2 mm to (11.0, 27.0), turned to 0 degrees
- moved C2 23.8 mm to (65.0, 37.0), turned to 180 degrees
- moved C26 22.3 mm to (24.0, 7.00), turned to 90 degrees
- moved C13 19.9 mm to (33.0, 19.5)
- moved C23 19.1 mm to (33.0, 11.0)
- moved C3 18.8 mm to (65.0, 13.2)
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- renumbered R30 to R29
Connections:
- net N$38 renamed SMBDAT
- net N$43 renamed SMBCLK
- net N$68 renamed USB_P
- net N$69 renamed USB_N
- net +1.8V: now also C12.2, C17.2, C21.2, C24.2, C26.2; no longer C13.2, C18.2, C22.2, C25.2, C27.2
- net +15V: now also C2.+, C4.2; no longer C1.+, C3.2
- net +3.3V: now also C10.+, C11.2, C14.2, C16.2, C19.2, C23.2, C28.2, C33.2; no longer C10.2, C15.2, C17.2, C21.2, C24.2, C29.2, C35.2, C5.+
- net -15V: now also C3.-, C5.1; no longer C2.-, C4.1
- net DGND: now also C1.-, C10.-, C11.1, C12.1, C33.1; no longer C10.1, C29.1, C35.1, C38.-, C5.-
- net GND: now also C2.-, C3.+, C4.1, C5.2; no longer C1.-, C2.+, C3.1, C4.2
- net N$10: now also C29.2, C30.-; no longer C30.2, C31.-
- net N$11: now also C36.2; no longer C37.2
- net N$12: now also C35.2; no longer C36.2
- net N$13: now also C35.1; no longer C36.1
- net N$14: now also C36.1; no longer C37.1
- net N$29: now also C1.+; no longer C38.+
- net N$36: now also C25.2, C31.1, C32.+; no longer C26.2, C32.1, C33.+
- net N$54: now also C13.2; no longer C14.2
- net N$56: now also C15.2; no longer C16.2
- net N$60: now also C18.2; no longer C19.2
- net N$62: now also C22.2; no longer C23.2
- net N$7: now also C27.2, C29.1, C30.+; no longer C28.2, C30.1, C31.+
- net N$9: now also C31.2, C32.-; no longer C32.2, C33.-
Routing:
- net DGND: track 13.3 -> 251.3 mm, vias 15 -> 31
- net GND: track 0.00 -> 157.0 mm, vias 0 -> 8
- net N$11: track 50.1 -> 35.5 mm, vias 0 -> 1
- net N$10: track 44.5 -> 30.0 mm, vias 0 -> 2
- net N$9: track 43.3 -> 29.5 mm, vias 0 -> 2
- net N$12: track 32.4 -> 40.6 mm
- net SMBCLK: track 84.2 -> 91.6 mm, vias 2 -> 1
- net N$44: track 37.3 -> 31.5 mm, vias 2 -> 3
- net -15V: track 33.0 -> 27.7 mm
- net N$39: track 18.7 -> 13.8 mm
- net N$7: track 27.2 -> 23.1 mm
- net SMBDAT: track 85.0 -> 88.5 mm
- net N$40: track 27.0 -> 24.5 mm
- net +3.3V: track 165.1 -> 167.4 mm, vias 10 -> 8
- net +1.8V: track 64.2 -> 66.1 mm, vias 5 -> 6
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
Commit message: PCB Update
Parts:
- removed O1: (no value), text:EMPTY
- added U10, U11, U8, U9: NUT-M2-SELFLOCK, hardware:EMPTY
- added U4, U5, U6, U7: SCREW-M2X8, hardware:EMPTY
- PCB1: value rev.A -> D709 rev.A
Changed lines of the file:
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@@
 <?xml version="1.0" encoding="utf-8"?>
 <!DOCTYPE eagle SYSTEM "eagle.dtd">
-<eagle version="7.5.0">
+<eagle version="7.5.1">
 <drawing>
 <settings>
@@
 </autorouter>
 <elements>
-<element name="O1" library="text" package="EMPTY" value="" x="81" y="-100"/>
-<element name="PCB1" library="module-footprints" package="ST2-BOARD-50" value="rev.A" x="0" y="0"/>
+<element name="PCB1" library="module-footprints" package="ST2-BOARD-50" value="D709 rev.A" x="0" y="0"/>
 <element name="C2" library="capacitors-electrolytic" package="E2-5" value="10U/35V" x="65" y="37" rot="R180">
 <attribute name="MOUSER" value="647-USW1V100MDD" x="94" y="18" size="1.778" layer="27" rot="R180" display="off"/>
@@
 <attribute name="MOUSER" value="647-USW1V100MDD" x="29" y="43" size="1.778" layer="27" rot="R270" display="off"/>
 </element>
+<element name="U4" library="hardware" package="EMPTY" value="SCREW-M2X8" x="-8" y="-104.25"/>
+<element name="U5" library="hardware" package="EMPTY" value="SCREW-M2X8" x="-9" y="-105.5"/>
+<element name="U6" library="hardware" package="EMPTY" value="SCREW-M2X8" x="-10" y="-106.75"/>
+<element name="U7" library="hardware" package="EMPTY" value="SCREW-M2X8" x="-11" y="-108"/>
+<element name="U8" library="hardware" package="EMPTY" value="NUT-M2-SELFLOCK" x="-12" y="-109.25"/>
+<element name="U9" library="hardware" package="EMPTY" value="NUT-M2-SELFLOCK" x="-13" y="-110.5"/>
+<element name="U10" library="hardware" package="EMPTY" value="NUT-M2-SELFLOCK" x="-14" y="-111.75"/>
+<element name="U11" library="hardware" package="EMPTY" value="NUT-M2-SELFLOCK" x="-15" y="-113"/>
 </elements>
 <signals>
