File: d701-vs1053-synth.sch (EAGLE design)
At the start: 88 parts, among them U1 FX2-20P-1.27DS, U2 FX2-20S-1.27DS, U3 ERM1-5MM

Commit message: d701 routing update
Parts:
- removed C37: 22P, capacitors:22P
- removed C38: 10U/35V, capacitors-electrolytic:10U/35V
- added C11, C12: 1U, capacitors:1U
- C10: value 1U -> 10U/35V; device capacitors:1U -> capacitors-electrolytic:10U/35V
- C14: value 1U -> 100N; device capacitors:1U -> capacitors:100N
- C15: value 100N -> 47N(FILM); device capacitors:100N -> capacitors:47N(FILM)
- C16: value 47N(FILM) -> 100N; device capacitors:47N(FILM) -> capacitors:100N
- C18, C22: value 100N -> 10N(FILM); device capacitors:100N -> capacitors:10N(FILM)
- C19, C23: value 10N(FILM) -> 100N; device capacitors:10N(FILM) -> capacitors:100N
- C25, C27: value 100N -> 3N3(FILM); device capacitors:100N -> capacitors:3N3(FILM)
- C26, C28: value 3N3(FILM) -> 100N; device capacitors:3N3(FILM) -> capacitors:100N
- C29: value 100N -> 100N(FILM); device capacitors:100N -> capacitors:100N(FILM)
- C3: value 100N -> 10U/35V; device capacitors:100N -> capacitors-electrolytic:10U/35V
- C30, C32: value 100N(FILM) -> 33U/25V; device capacitors:100N(FILM) -> capacitors-electrolytic:33U/25V
- C31: value 47U/35V -> 100N(FILM); device capacitors-electrolytic:47U/35V -> capacitors:100N(FILM)
- C33: value 47U/35V -> 100N; device capacitors-electrolytic:47U/35V -> capacitors:100N
- C35: value 100N -> 22P; device capacitors:100N -> capacitors:22P
- C5: value 10U/35V -> 100N; device capacitors-electrolytic:10U/35V -> capacitors:100N
- renumbered R30 to R29
Connections:
- net N$38 renamed SMBDAT
- net N$43 renamed SMBCLK
- net N$68 renamed USB_P
- net N$69 renamed USB_N
- net +1.8V: now also C12.2, C17.2, C21.2, C24.2, C26.2; no longer C13.2, C18.2, C22.2, C25.2, C27.2
- net +15V: now also C2.+, C4.2; no longer C1.+, C3.2
- net +3.3V: now also C10.+, C11.2, C14.2, C16.2, C19.2, C23.2, C28.2, C33.2; no longer C10.2, C15.2, C17.2, C21.2, C24.2, C29.2, C35.2, C5.+
- net -15V: now also C3.-, C5.1; no longer C2.-, C4.1
- net DGND: now also C1.-, C10.-, C11.1, C12.1, C33.1; no longer C10.1, C29.1, C35.1, C38.-, C5.-
- net GND: now also C2.-, C3.+, C4.1, C5.2; no longer C1.-, C2.+, C3.1, C4.2
- net N$10: now also C29.2, C30.-; no longer C30.2, C31.-
- net N$11: now also C36.2; no longer C37.2
- net N$12: now also C35.2; no longer C36.2
- net N$13: now also C35.1; no longer C36.1
- net N$14: now also C36.1; no longer C37.1
- net N$29: now also C1.+; no longer C38.+
- net N$36: now also C25.2, C31.1, C32.+; no longer C26.2, C32.1, C33.+
- net N$54: now also C13.2; no longer C14.2
- net N$56: now also C15.2; no longer C16.2
- net N$60: now also C18.2; no longer C19.2
- net N$62: now also C22.2; no longer C23.2
- net N$7: now also C27.2, C29.1, C30.+; no longer C28.2, C30.1, C31.+
- net N$9: now also C31.2, C32.-; no longer C32.2, C33.-
Other:
- moved on the sheet: C1, C13, C14, C15, C16, C17, C18, C19, C2, C20, C21, C22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

Commit message: PCB Update
Parts:
- removed O1: (no value), text:TITLE
- added U10, U11, U8, U9: NUT-M2-SELFLOCK, hardware:NUT-M2-SELFLOCK
- added U4, U5, U6, U7: SCREW-M2X8, hardware:SCREW-M2X8
- PCB1: value rev.A -> D709 rev.A
Other:
- moved on the sheet: U1, U2
Changed lines of the file:
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@@
 <?xml version="1.0" encoding="utf-8"?>
 <!DOCTYPE eagle SYSTEM "eagle.dtd">
-<eagle version="7.5.0">
+<eagle version="7.5.1">
 <drawing>
 <settings>
@@
 </classes>
 <parts>
-<part name="O1" library="text" deviceset="TITLE" device=""/>
-<part name="PCB1" library="module-footprints" deviceset="ST2-BOARD-?" device="50" value="rev.A"/>
+<part name="PCB1" library="module-footprints" deviceset="ST2-BOARD-?" device="50" value="D709 rev.A"/>
 <part name="C2" library="capacitors-electrolytic" deviceset="?" device="10U/35V" value="10U/35V"/>
 <part name="C3" library="capacitors-electrolytic" deviceset="?" device="10U/35V" value="10U/35V"/>
@@
 <part name="C1" library="capacitors-electrolytic" deviceset="?" device="10U/35V" value="10U/35V"/>
 <part name="GND3" library="supply" deviceset="DGND" device=""/>
+<part name="U4" library="hardware" deviceset="*?" device="SCREW-M2X8"/>
+<part name="U5" library="hardware" deviceset="*?" device="SCREW-M2X8"/>
+<part name="U6" library="hardware" deviceset="*?" device="SCREW-M2X8"/>
+<part name="U7" library="hardware" deviceset="*?" device="SCREW-M2X8"/>
+<part name="U8" library="hardware" deviceset="*?" device="NUT-M2-SELFLOCK"/>
+<part name="U9" library="hardware" deviceset="*?" device="NUT-M2-SELFLOCK"/>
+<part name="U10" library="hardware" deviceset="*?" device="NUT-M2-SELFLOCK"/>
+<part name="U11" library="hardware" deviceset="*?" device="NUT-M2-SELFLOCK"/>
 </parts>
 <sheets>
@@
 </plain>
 <instances>
-<instance part="O1" gate="G$1" x="-5.08" y="358.14"/>
-<instance part="PCB1" gate="G$1" x="88.9" y="360.68"/>
+<instance part="PCB1" gate="G$1" x="15.24" y="360.68"/>
 <instance part="PCB1" gate="G$2" x="7.62" y="335.28"/>
 <instance part="PCB1" gate="G$3" x="7.62" y="330.2"/>
@@
 <instance part="GND2" gate="VR1" x="53.34" y="276.86"/>
 <instance part="GND4" gate="VR1" x="58.42" y="276.86"/>
-<instance part="U1" gate="G$1" x="81.28" y="332.74"/>
-<instance part="U2" gate="G$1" x="81.28" y="325.12"/>
+<instance part="U1" gate="G$1" x="58.42" y="360.68"/>
+<instance part="U2" gate="G$1" x="88.9" y="360.68"/>
 <instance part="DD3" gate="G$1" x="132.08" y="132.08"/>
 <instance part="DD2" gate="G$1" x="132.08" y="231.14"/>
@@
 </instance>
 <instance part="GND3" gate="1" x="55.88" y="35.56"/>
+<instance part="U4" gate="G$1" x="48.26" y="353.06"/>
+<instance part="U5" gate="G$1" x="48.26" y="350.52"/>
+<instance part="U6" gate="G$1" x="78.74" y="353.06"/>
+<instance part="U7" gate="G$1" x="78.74" y="350.52"/>
+<instance part="U8" gate="G$1" x="48.26" y="347.98"/>
+<instance part="U9" gate="G$1" x="48.26" y="345.44"/>
+<instance part="U10" gate="G$1" x="78.74" y="347.98"/>
+<instance part="U11" gate="G$1" x="78.74" y="345.44"/>
 </instances>
 <busses>
@@
 </schematic>
 </drawing>
-<compatibility>
-<note version="6.3" minversion="6.2.2" severity="warning">
-Since Version 6.2.2 text objects can contain more than one line,
-which will not be processed correctly with this version.
-</note>
-</compatibility>
 </eagle>
