File: d101-lofi-delay.brd (EAGLE design)
At the start: 100 x 50 mm, 84 parts, among them U1 FX2-20P-1.27DS, U2 FX2-20S-1.27DS

Commit message: Add Knobs
Parts:
- added O2, O3, O4: 450-AA150(15MM,D,BLACK), hardware:EMPTY
- added O5: 450-CP155(15MM,GRAY/WHITE), hardware:EMPTY
- added O6, O7: 450-CP157(15MM,WHITE/BLACK), hardware:EMPTY
Changed lines of the file:
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@@
 <?xml version="1.0" encoding="utf-8"?>
 <!DOCTYPE eagle SYSTEM "eagle.dtd">
-<eagle version="7.4.1">
+<eagle version="7.5.1">
 <drawing>
 <settings>
@@
 <attribute name="MOUSER" value="642-MJS22R" x="0" y="25" size="1.778" layer="27" rot="R90" display="off"/>
 </element>
+<element name="O2" library="hardware" package="EMPTY" value="450-AA150(15MM,D,BLACK)" x="-62" y="-10.25">
+<attribute name="MOUSER" value="450-AA150" x="-62" y="-10.25" size="1.778" layer="27" display="off"/>
+</element>
+<element name="O3" library="hardware" package="EMPTY" value="450-AA150(15MM,D,BLACK)" x="-63" y="-11.5">
+<attribute name="MOUSER" value="450-AA150" x="-63" y="-11.5" size="1.778" layer="27" display="off"/>
+</element>
+<element name="O4" library="hardware" package="EMPTY" value="450-AA150(15MM,D,BLACK)" x="-64" y="-12.75">
+<attribute name="MOUSER" value="450-AA150" x="-64" y="-12.75" size="1.778" layer="27" display="off"/>
+</element>
+<element name="O5" library="hardware" package="EMPTY" value="450-CP155(15MM,GRAY/WHITE)" x="-65" y="-14">
+<attribute name="MOUSER" value="450-CP155" x="-65" y="-14" size="1.778" layer="27" display="off"/>
+</element>
+<element name="O6" library="hardware" package="EMPTY" value="450-CP157(15MM,WHITE/BLACK)" x="-66" y="-15.25">
+<attribute name="MOUSER" value="450-CP157" x="-66" y="-15.25" size="1.778" layer="27" display="off"/>
+</element>
+<element name="O7" library="hardware" package="EMPTY" value="450-CP157(15MM,WHITE/BLACK)" x="-67" y="-16.5">
+<attribute name="MOUSER" value="450-CP157" x="-67" y="-16.5" size="1.778" layer="27" display="off"/>
+</element>
 </elements>

Commit message: Add Knobs
Parts:
- removed C34, C35: 100N, capacitors:C-0805
- removed C36, C37: 47N(FILM), capacitors:C050-025X075
- removed C38, C39: 33U/25V, capacitors-electrolytic:E2,5-7
- removed O7: 450-CP157(15MM,WHITE/BLACK), hardware:EMPTY
- removed R36, R37, R38, R39: 10K, resistors:R-0805
- removed R41, R43, R44, R45: 1K, resistors:R-0805
- added C10, C11: 10N(FILM), capacitors:C050-025X075
- added C12, C13: 100N, capacitors:C-0805
- added C8, C9: 100N(FILM), capacitors:C050-025X075
- added R12, R13, R22, R23: 15K, resistors:R-0805
- added R14: 1K, resistors:R-0805
- added R21, R24, R25: 10K, resistors:R-0805
- added U10: FX2-20S-1.27DS, hardware:EMPTY
- added U11, U12: D-SHAFT-ADAPTER, hardware:EMPTY
- added U3, U4, U8, U9: NUT-M2-SELFLOCK, hardware:EMPTY
- added U5: FX2-20P-1.27DS, hardware:EMPTY
- added U6, U7: SCREW-M2X8, hardware:EMPTY
- C14, C15: value 100N(FILM) -> 2N2(FILM)
- C16, C17: value 10N(FILM) -> 10U/35V; device capacitors:C050-025X075 -> capacitors-electrolytic:E2-5
- C18, C19: value 100N -> 2N2(FILM); device capacitors:C-0805 -> capacitors:C050-025X075
- C20, C21: value 2N2(FILM) -> 100N(FILM)
- C22, C23: value 10U/35V -> 10N(FILM); device capacitors-electrolytic:E2-5 -> capacitors:C050-025X075
- C24, C25: value 2N2(FILM) -> 100N; device capacitors:C050-025X075 -> capacitors:C-0805
- C28, C29: value 10N(FILM) -> 100N; device capacitors:C050-025X075 -> capacitors:C-0805
- C30, C31: value 100N -> 47N(FILM); device capacitors:C-0805 -> capacitors:C050-025X075
- C32, C33: value 100N(FILM) -> 33U/25V; device capacitors:C050-025X075 -> capacitors-electrolytic:E2,5-7
- O1: value (none) -> 450-AA150(15MM,D,BLACK); device text:EMPTY -> hardware:EMPTY
- O2: value 450-AA150(15MM,D,BLACK) -> 450-CP155(15MM,GRAY/WHITE)
- O4: value 450-AA150(15MM,D,BLACK) -> 450-CP157(15MM,WHITE/BLACK)
- O5: value 450-CP155(15MM,GRAY/WHITE) -> 450-AA150(15MM,D,BLACK)
- PCB1: value rev.A -> D101 rev.A
- R15, R32: value 15K -> 1K
- R16: value 15K -> 100K
- R17: value 1K -> 100K
- R18: value 1K -> 10K
- R19, R20: value B50K** -> 10K; device potentiometers:RV11-SINGLE -> resistors:R-0805
- R26, R27: value 100K -> 10K
- R30, R34, R35: value 10K -> 1K
- R31: value 10K -> B50K**; device resistors:R-0805 -> potentiometers:RV11-SINGLE
- R33: value 15K -> B50K**; device resistors:R-0805 -> potentiometers:RV11-SINGLE
- U1: value FX2-20P-1.27DS -> SCREW-M2X8
- U2: value FX2-20S-1.27DS -> SCREW-M2X8
- moved O1 111.6 mm to (-62.0, -10.2)
- moved C32 45.1 mm to (20.5, 8.00)
- moved R31 40.1 mm to (82.8, 37.2), turned to 90 degrees
- moved R19 35.0 mm to (48.0, 13.0)
- moved C30 34.4 mm to (40.0, 33.0), turned to 0 degrees
- moved C31 34.0 mm to (40.0, 18.0), turned to 0 degrees
- moved R20 33.0 mm to (53.0, 23.0)
- moved R32 32.8 mm to (83.0, 23.0), turned to 180 degrees
- moved C33 32.7 mm to (28.0, 8.00), turned to 180 degrees
- moved C17 32.0 mm to (71.0, 7.00), turned to 180 degrees
- moved C16 31.3 mm to (71.0, 26.0)
- moved R33 31.0 mm to (83.0, 13.0), turned to 90 degrees
- moved R30 30.3 mm to (83.0, 27.0), turned to 180 degrees
- moved R16 28.2 mm to (48.0, 23.0), turned to 270 degrees
- moved R15 27.7 mm to (34.0, 32.0), turned to 0 degrees
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- renumbered SA2 to SA1
Connections:
- net +5V: now also C12.2, C13.2; no longer C18.2, C19.2
- net FBK_INT_LEFT: now also R12.2; no longer R15.2
- net FBK_INT_RIGHT: now also R13.2; no longer R16.2
- net GND: now also C10.1, C11.1, C12.1, C13.1, C16.-, C17.-, C22.1, C23.1, C24.1, C25.1, R16.1, R17.1, R31.2, R31.3, R33.2, R33.3, VD1.2, VD4.1; no longer C16.1, C17.1, C18.1, C19.1, C22.-, C23.-, C34.1, C35.1, C36.1, C37.1, R19.2, R19.3, R20.2, R20.3, R26.1, R27.1, VD1.1, VD4.2
- net N$1: now also R32.1, R33.1; no longer R19.1, R43.1
- net N$10: now also C11.2, R19.2, R21.2, R23.2; no longer C17.2, R29.2, R31.2, R33.2
- net N$13: now also R15.1; no longer R18.1
- net N$15: now also C23.2, R25.2, R27.2, R29.2; no longer C29.2, R35.2, R37.2, R39.2
- net N$17: now also C15.2, R23.1; no longer C21.2, R33.1
- net N$18: now also C19.1, R25.1; no longer C25.1, R45.1
- net N$19: now also C19.2, R27.1; no longer C25.2, R37.1
- net N$2: now also R30.1, R31.1; no longer R20.1, R41.1
- net N$20: now also C21.1, R29.1; no longer C27.1, R39.1
- net N$21: now also C21.2; no longer C27.2
- net N$22: now also C27.1; no longer C33.1
- net N$23: now also C27.2; no longer C33.2
- net N$24: now also C31.2, C33.+, R35.2; no longer C37.2, C39.+, R45.2
- net N$25: now also R13.1; no longer R16.1
- net N$28: now also R3.1; no longer R7.1
- net N$3: now also C9.1, R14.2, VD1.1, VD3.2; no longer C15.1, R17.2, VD1.2, VD2.1
- net N$30: now also R7.1; no longer R2.1
- net N$31: now also C25.2; no longer C31.2
- net N$32: now also C29.2; no longer C35.2
- net N$33: now also R32.2; no longer R43.2
- net N$37: now also C17.+; no longer C23.+
- net N$39: now also R10.2; no longer R8.2
- net N$4: now also C15.1, R21.1; no longer C21.1, R31.1
- net N$40: now also R4.2; no longer R10.2
- net N$48: now also C22.2, R24.2, R26.2, R28.2; no longer C28.2, R34.2, R36.2, R38.2
- net N$49: now also C14.1, R20.1; no longer C20.1, R30.1
- net N$5: now also C8.1, R15.2, VD2.1, VD4.2; no longer C14.1, R18.2, VD3.2, VD4.1
- net N$50: now also C14.2, R22.1; no longer C20.2, R32.1
- net N$51: now also C18.1, R24.1; no longer C24.1, R44.1
- net N$52: now also C18.2, R26.1; no longer C24.2, R36.1
- net N$53: now also C20.1, R28.1; no longer C26.1, R38.1
- net N$54: now also C20.2; no longer C26.2
- net N$55: now also C26.1; no longer C32.1
- net N$56: now also C26.2; no longer C32.2
- net N$57: now also C30.2, C32.+, R34.2; no longer C36.2, C38.+, R44.2
- net N$58: now also C24.2; no longer C30.2
- net N$59: now also C28.2; no longer C34.2
- net N$6: now also R14.1; no longer R17.1
- net N$60: now also R30.2; no longer R41.2
- net N$61: now also R7.2, R8.2; no longer R2.2, R4.2
- net N$62: now also C8.2, R16.2, R18.1; no longer C14.2, R26.2, R28.1
- net N$63: now also C10.2, R18.2, R20.2, R22.2; no longer C16.2, R28.2, R30.2, R32.2
- net N$64: now also R12.1; no longer R15.1
- net N$65: now also R2.2, R8.1; no longer R3.2, R4.1
- net N$69: now also C16.+; no longer C22.+
- net N$7: now also R10.1, R3.2; no longer R7.2, R8.1
- net N$9: now also C9.2, R17.2, R19.1; no longer C15.2, R27.2, R29.1
- net OUT_LEFT: now also C33.-, R4.1; no longer C39.-, R10.1
- net OUT_RIGHT: now also C32.-, R2.1; no longer C38.-, R3.1

Commit message: D101 Update
Parts:
- added R36, R37: 1K, resistors:R-0805
- R28, R29: value 10K -> 100K
- R30: value 1K -> 10K
- R31: value B50K** -> 10K; device potentiometers:RV11-SINGLE -> resistors:R-0805
- R33: value B50K** -> B100K
- R35: value 1K -> B100K; device resistors:R-0805 -> potentiometers:RV11-SINGLE
- moved R34 36.5 mm to (83.0, 23.0)
- moved R35 35.4 mm to (83.0, 13.0)
- moved R33 24.3 mm to (82.8, 37.2)
- moved R28 22.7 mm to (87.5, 27.0), turned to 180 degrees
- moved R31 21.6 mm to (67.5, 22.0), turned to 180 degrees
- moved R29 20.0 mm to (87.5, 23.0)
- moved R30 19.5 mm to (70.5, 42.0), turned to 270 degrees
- moved R32 4.00 mm to (83.0, 27.0)
Connections:
- net GND: now also R28.1, R29.1, R35.2, R35.3; no longer R31.2, R31.3
- net N$1: now also R29.2, R34.1, R35.1; no longer R32.1, R33.1
- net N$15: now also R31.2; no longer R29.2
- net N$18: now also R37.1; no longer R35.1
- net N$2: now also R28.2, R32.1, R33.1; no longer R30.1, R31.1
- net N$20: now also R31.1; no longer R29.1
- net N$24: now also R37.2; no longer R35.2
- net N$33: now also R34.2; no longer R32.2
- net N$48: now also R30.2; no longer R28.2
- net N$51: now also R36.1; no longer R34.1
- net N$53: now also R30.1; no longer R28.1
- net N$57: now also R36.2; no longer R34.2
- net N$60: now also R32.2; no longer R30.2
Routing:
- net N$1: track 18.7 -> 20.9 mm
- net N$2: track 12.4 -> 12.9 mm

Commit message: PCB Update
Parts:
- removed U11, U12: D-SHAFT-ADAPTER, hardware:EMPTY
- PCB1: value D101 rev.A -> D104 rev.A
Changed lines of the file:
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@@
 </autorouter>
 <elements>
-<element name="PCB1" library="module-footprints" package="ST2-BOARD-50" value="D101 rev.A" x="0" y="0" smashed="yes">
+<element name="PCB1" library="module-footprints" package="ST2-BOARD-50" value="D104 rev.A" x="0" y="0" smashed="yes">
 <attribute name="VALUE" x="98" y="25" size="1.27" layer="21" ratio="15" rot="R270" align="bottom-center"/>
 </element>
@@
 <element name="U8" library="hardware" package="EMPTY" value="NUT-M2-SELFLOCK" x="-74" y="-25.25"/>
 <element name="U9" library="hardware" package="EMPTY" value="NUT-M2-SELFLOCK" x="-75" y="-26.5"/>
-<element name="U12" library="hardware" package="EMPTY" value="D-SHAFT-ADAPTER" x="-76" y="-27.75"/>
-<element name="U11" library="hardware" package="EMPTY" value="D-SHAFT-ADAPTER" x="-77" y="-29"/>
 <element name="R29" library="resistors" package="R-0805" value="100K" x="87.5" y="23" rot="R180">
 <attribute name="MOUSER" value="660-RK73H2ATTD1003F" x="87.5" y="23" size="1.778" layer="27" rot="R180" display="off"/>
