File: d102-spinsemi-fx.brd (EAGLE design)
At the start: 100 x 50 mm, 74 parts, among them U1 FX2-20P-1.27DS, U2 FX2-20S-1.27DS, U3 ERM1-5MM

Commit message: PCB Update
Parts:
- removed O1: (no value), text:EMPTY
- added U10, U11, U8, U9: NUT-M2-SELFLOCK, hardware:EMPTY
- added U4, U5, U6, U7: SCREW-M2X8, hardware:EMPTY
- PCB1: value rev.A -> D108 rev.A
Changed lines of the file:
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@@
 <?xml version="1.0" encoding="utf-8"?>
 <!DOCTYPE eagle SYSTEM "eagle.dtd">
-<eagle version="7.4.1">
+<eagle version="7.5.1">
 <drawing>
 <settings>
@@
 </autorouter>
 <elements>
-<element name="O1" library="text" package="EMPTY" value="" x="9" y="-89"/>
-<element name="PCB1" library="module-footprints" package="ST2-BOARD-50" value="rev.A" x="0" y="0"/>
+<element name="PCB1" library="module-footprints" package="ST2-BOARD-50" value="D108 rev.A" x="0" y="0"/>
 <element name="U1" library="hardware" package="EMPTY" value="FX2-20P-1.27DS" x="12" y="-89">
 <attribute name="MOUSER" value="798-FX2-20P-1.27DS71" x="-1" y="-63" size="1.778" layer="27" display="off"/>
@@
 <attribute name="MOUSER" value="450-CP156" x="-76" y="-218" size="1.778" layer="27" display="off"/>
 </element>
+<element name="U4" library="hardware" package="EMPTY" value="SCREW-M2X8" x="-77" y="-219.25"/>
+<element name="U5" library="hardware" package="EMPTY" value="SCREW-M2X8" x="-78" y="-220.5"/>
+<element name="U6" library="hardware" package="EMPTY" value="SCREW-M2X8" x="-79" y="-221.75"/>
+<element name="U7" library="hardware" package="EMPTY" value="SCREW-M2X8" x="-80" y="-223"/>
+<element name="U8" library="hardware" package="EMPTY" value="NUT-M2-SELFLOCK" x="-81" y="-224.25"/>
+<element name="U9" library="hardware" package="EMPTY" value="NUT-M2-SELFLOCK" x="-82" y="-225.5"/>
+<element name="U10" library="hardware" package="EMPTY" value="NUT-M2-SELFLOCK" x="-83" y="-226.75"/>
+<element name="U11" library="hardware" package="EMPTY" value="NUT-M2-SELFLOCK" x="-84" y="-228"/>
 </elements>
 <signals>
