File: m901-vu-meter.brd (EAGLE design)
At the start: 100 x 26 mm, 46 parts, among them U1 ERM1-5MM, U10 ERM1-5MM, U11 ERM1-5MM, U12 ERM1-5MM, U2 ERM1-5MM, U3 FX2-20P-1.27DS, U4 FX2-20S-1.27DS, U5 ERM1-5MM, U6 ERM1-5MM, U7 ERM1-5MM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

Commit message: PCB Update
Parts:
- removed O1: (no value), text:EMPTY
- added U13, U14, U15, U16: SCREW-M2X8, hardware:EMPTY
- added U17, U18, U19, U20: NUT-M2-SELFLOCK, hardware:EMPTY
- PCB1: value rev.A -> M907 rev.A
Changed lines of the file:
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@@
 <?xml version="1.0" encoding="utf-8"?>
 <!DOCTYPE eagle SYSTEM "eagle.dtd">
-<eagle version="7.4.1">
+<eagle version="7.5.1">
 <drawing>
 <settings>
@@
 <attribute name="NAME" x="16" y="21.96" size="0.8128" layer="25" ratio="15" align="bottom-center"/>
 </element>
-<element name="O1" library="text" package="EMPTY" value="" x="-13.97" y="80.01"/>
-<element name="PCB1" library="module-footprints" package="ST2-BOARD-26" value="rev.A" x="0" y="0"/>
+<element name="PCB1" library="module-footprints" package="ST2-BOARD-26" value="M907 rev.A" x="0" y="0"/>
 <element name="R1" library="potentiometers" package="64W" value="10K(64W/Y)" x="72" y="7.5" smashed="yes" rot="R270">
 <attribute name="MOUSER" value="858-64WR10KLF" x="72" y="7.5" size="1.778" layer="27" rot="R270" display="off"/>
@@
 <element name="U11" library="hardware" package="EMPTY" value="ERM1-5MM" x="-28" y="-23"/>
 <element name="U12" library="hardware" package="EMPTY" value="ERM1-5MM" x="-29" y="-25"/>
+<element name="U13" library="hardware" package="EMPTY" value="SCREW-M2X8" x="-30" y="-26.25"/>
+<element name="U14" library="hardware" package="EMPTY" value="SCREW-M2X8" x="-31" y="-27.5"/>
+<element name="U15" library="hardware" package="EMPTY" value="SCREW-M2X8" x="-32" y="-28.75"/>
+<element name="U16" library="hardware" package="EMPTY" value="SCREW-M2X8" x="-33" y="-30"/>
+<element name="U17" library="hardware" package="EMPTY" value="NUT-M2-SELFLOCK" x="-34" y="-31.25"/>
+<element name="U18" library="hardware" package="EMPTY" value="NUT-M2-SELFLOCK" x="-35" y="-32.5"/>
+<element name="U19" library="hardware" package="EMPTY" value="NUT-M2-SELFLOCK" x="-36" y="-33.75"/>
+<element name="U20" library="hardware" package="EMPTY" value="NUT-M2-SELFLOCK" x="-37" y="-35"/>
 </elements>
 <signals>
