File: m901-vu-meter.sch (EAGLE design)
At the start: 46 parts, among them U1 ERM1-5MM, U10 ERM1-5MM, U11 ERM1-5MM, U12 ERM1-5MM, U2 ERM1-5MM, U3 FX2-20P-1.27DS, U4 FX2-20S-1.27DS, U5 ERM1-5MM, U6 ERM1-5MM, U7 ERM1-5MM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

Commit message: PCB Update
Parts:
- removed O1: (no value), text:TITLE
- added U13, U14, U15, U16: SCREW-M2X8, hardware:SCREW-M2X8
- added U17, U18, U19, U20: NUT-M2-SELFLOCK, hardware:NUT-M2-SELFLOCK
- PCB1: value rev.A -> M907 rev.A
Other:
- moved on the sheet: U3, U4
Changed lines of the file:
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@@
 <?xml version="1.0" encoding="utf-8"?>
 <!DOCTYPE eagle SYSTEM "eagle.dtd">
-<eagle version="7.4.1">
+<eagle version="7.5.1">
 <drawing>
 <settings>
@@
 </classes>
 <parts>
-<part name="O1" library="text" deviceset="TITLE" device=""/>
-<part name="PCB1" library="module-footprints" deviceset="ST2-BOARD-?" device="26" value="rev.A"/>
+<part name="PCB1" library="module-footprints" deviceset="ST2-BOARD-?" device="26" value="M907 rev.A"/>
 <part name="L1" library="inductors" deviceset="BL01RN1A?" device="1F1J"/>
 <part name="C5" library="capacitors-electrolytic" deviceset="?" device="10U/35V" value="10U/35V"/>
@@
 <part name="U11" library="hardware" deviceset="?" device="ERM1-5MM"/>
 <part name="U12" library="hardware" deviceset="?" device="ERM1-5MM"/>
+<part name="U13" library="hardware" deviceset="*?" device="SCREW-M2X8"/>
+<part name="U14" library="hardware" deviceset="*?" device="SCREW-M2X8"/>
+<part name="U15" library="hardware" deviceset="*?" device="SCREW-M2X8"/>
+<part name="U16" library="hardware" deviceset="*?" device="SCREW-M2X8"/>
+<part name="U17" library="hardware" deviceset="*?" device="NUT-M2-SELFLOCK"/>
+<part name="U18" library="hardware" deviceset="*?" device="NUT-M2-SELFLOCK"/>
+<part name="U19" library="hardware" deviceset="*?" device="NUT-M2-SELFLOCK"/>
+<part name="U20" library="hardware" deviceset="*?" device="NUT-M2-SELFLOCK"/>
 </parts>
 <sheets>
@@
 </plain>
 <instances>
-<instance part="O1" gate="G$1" x="0" y="231.14"/>
-<instance part="PCB1" gate="G$1" x="93.98" y="233.68"/>
+<instance part="PCB1" gate="G$1" x="20.32" y="213.36"/>
 <instance part="PCB1" gate="G$2" x="12.7" y="147.32"/>
 <instance part="PCB1" gate="G$3" x="12.7" y="104.14"/>
@@
 <instance part="PCB1" gate="G$8" x="12.7" y="157.48"/>
 <instance part="PCB1" gate="G$9" x="12.7" y="35.56"/>
-<instance part="U3" gate="G$1" x="86.36" y="205.74"/>
-<instance part="U4" gate="G$1" x="86.36" y="198.12"/>
+<instance part="U3" gate="G$1" x="58.42" y="213.36"/>
+<instance part="U4" gate="G$1" x="86.36" y="213.36"/>
 <instance part="C1" gate="G$1" x="81.28" y="35.56" smashed="yes" rot="R270">
 <attribute name="NAME" x="79.248" y="35.56" size="1.778" layer="94" rot="R90" align="bottom-center"/>
@@
 <instance part="U11" gate="G$1" x="149.86" y="76.2"/>
 <instance part="U12" gate="G$1" x="149.86" y="68.58"/>
+<instance part="U13" gate="G$1" x="48.26" y="205.74"/>
+<instance part="U14" gate="G$1" x="48.26" y="203.2"/>
+<instance part="U15" gate="G$1" x="76.2" y="205.74"/>
+<instance part="U16" gate="G$1" x="76.2" y="203.2"/>
+<instance part="U17" gate="G$1" x="48.26" y="200.66"/>
+<instance part="U18" gate="G$1" x="48.26" y="198.12"/>
+<instance part="U19" gate="G$1" x="76.2" y="200.66"/>
+<instance part="U20" gate="G$1" x="76.2" y="198.12"/>
 </instances>
 <busses>
@@
 </schematic>
 </drawing>
-<compatibility>
-<note version="6.3" minversion="6.2.2" severity="warning">
-Since Version 6.2.2 text objects can contain more than one line,
-which will not be processed correctly with this version.
-</note>
-</compatibility>
 </eagle>
