File: m2101-psu-dcdc.sch (EAGLE design)
At the start: 36 parts, among them U1 FX2-20P-1.27DS, U2 SHHN000A3CL41Z, U3 G3VM-62C1, U4 ERM1-5MM

Commit message: Board rev.A -> rev.B
Parts:
- PCB1: value rev.A -> rev.B
Changed lines of the file:
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@@
 <part name="O1" library="text" deviceset="TITLE" device="" value="Designed by Artem Godin // fluorumlabs.com"/>
 <part name="XS1" library="connectors" deviceset="PJ-051?" device="AH"/>
-<part name="PCB1" library="module-footprints" deviceset="ST2-BOARD-50-PSU" device="" value="rev.A"/>
+<part name="PCB1" library="module-footprints" deviceset="ST2-BOARD-50-PSU" device="" value="rev.B"/>
 <part name="GND1" library="supply" deviceset="GND" device=""/>
 <part name="VD1" library="diodes" deviceset="DF?M" device="01"/>

Commit message: PSU PCB Update
Parts:
- removed O1: Designed by Artem Godin // fluorumlabs.com, text:TITLE
- added U5, U6: SCREW-M2X8, hardware:SCREW-M2X8
- added U7, U8: NUT-M2-SELFLOCK, hardware:NUT-M2-SELFLOCK
- PCB1: value rev.B -> M101 rev.B
Other:
- moved on the sheet: U1
Changed lines of the file:
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@@
 <?xml version="1.0" encoding="utf-8"?>
 <!DOCTYPE eagle SYSTEM "eagle.dtd">
-<eagle version="7.5.0">
+<eagle version="7.5.1">
 <drawing>
 <settings>
@@
 <variant name="+15V/0/-15V Input" populate="no"/>
 </part>
-<part name="O1" library="text" deviceset="TITLE" device="" value="Designed by Artem Godin // fluorumlabs.com"/>
 <part name="XS1" library="connectors" deviceset="PJ-051?" device="AH"/>
-<part name="PCB1" library="module-footprints" deviceset="ST2-BOARD-50-PSU" device="" value="rev.B"/>
+<part name="PCB1" library="module-footprints" deviceset="ST2-BOARD-50-PSU" device="" value="M101 rev.B"/>
 <part name="GND1" library="supply" deviceset="GND" device=""/>
 <part name="VD1" library="diodes" deviceset="DF?M" device="01"/>
@@
 <part name="SA1" library="switches" deviceset="MHS122K" device=""/>
 <part name="S1" library="switches" deviceset="JUMPER-1POS-SOLDER" device=""/>
+<part name="U5" library="hardware" deviceset="*?" device="SCREW-M2X8"/>
+<part name="U6" library="hardware" deviceset="*?" device="SCREW-M2X8"/>
+<part name="U7" library="hardware" deviceset="*?" device="NUT-M2-SELFLOCK"/>
+<part name="U8" library="hardware" deviceset="*?" device="NUT-M2-SELFLOCK"/>
 </parts>
 <sheets>
@@
 <attribute name="VALUE" x="45.72" y="-111.76" size="1.778" layer="96" align="bottom-center"/>
 </instance>
-<instance part="O1" gate="G$1" x="55.88" y="0"/>
 <instance part="XS1" gate="G$1" x="-2.54" y="-93.98"/>
-<instance part="PCB1" gate="G$1" x="137.16" y="2.54"/>
+<instance part="PCB1" gate="G$1" x="73.66" y="2.54"/>
 <instance part="PCB1" gate="G$2" x="5.08" y="2.54" rot="MR0"/>
 <instance part="PCB1" gate="G$3" x="5.08" y="-2.54" rot="MR0"/>
@@
 <instance part="R8" gate="G$1" x="195.58" y="-132.08" rot="R90"/>
 <instance part="R9" gate="G$1" x="215.9" y="-132.08" rot="R90"/>
-<instance part="U1" gate="G$1" x="5.08" y="-48.26"/>
+<instance part="U1" gate="G$1" x="111.76" y="2.54"/>
 <instance part="U3" gate=".1A" x="144.78" y="-40.64" rot="R270"/>
 <instance part="U3" gate=".2A" x="132.08" y="-40.64" rot="R270"/>
@@
 <instance part="SA1" gate=".2" x="93.98" y="-99.06" rot="MR0"/>
 <instance part="S1" gate="G$1" x="93.98" y="-114.3"/>
+<instance part="U5" gate="G$1" x="101.6" y="-5.08"/>
+<instance part="U6" gate="G$1" x="101.6" y="-7.62"/>
+<instance part="U7" gate="G$1" x="101.6" y="-10.16"/>
+<instance part="U8" gate="G$1" x="101.6" y="-12.7"/>
 </instances>
 <busses>
@@
 </schematic>
 </drawing>
-<compatibility>
-<note version="6.3" minversion="6.2.2" severity="warning">
-Since Version 6.2.2 text objects can contain more than one line,
-which will not be processed correctly with this version.
-</note>
-</compatibility>
 </eagle>
