File: a405-diode-distortion.brd (EAGLE design)
At the start: 100 x 50 mm, 54 parts, among them U1 FX2-20P-1.27DS, U2 FX2-20S-1.27DS

Commit message: A405 Update
Parts:
- removed O1: (no value), text:EMPTY
- added U10, U7, U8, U9: NUT-M2-SELFLOCK, hardware:EMPTY
- added U3, U4, U5, U6: SCREW-M2X8, hardware:EMPTY
- PCB1: value rev.A -> A405 rev.A
Changed lines of the file:
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@@
 <?xml version="1.0" encoding="utf-8"?>
 <!DOCTYPE eagle SYSTEM "eagle.dtd">
-<eagle version="7.4.1">
+<eagle version="7.5.1">
 <drawing>
 <settings>
@@
 </autorouter>
 <elements>
-<element name="O1" library="text" package="EMPTY" value="" x="80" y="-99"/>
-<element name="PCB1" library="module-footprints" package="ST2-BOARD-50" value="rev.A" x="0" y="0"/>
+<element name="PCB1" library="module-footprints" package="ST2-BOARD-50" value="A405 rev.A" x="0" y="0"/>
 <element name="U1" library="hardware" package="EMPTY" value="FX2-20P-1.27DS" x="83" y="-99">
 <attribute name="MOUSER" value="798-FX2-20P-1.27DS71" x="-1" y="-63" size="1.778" layer="27" display="off"/>
@@
 <attribute name="MOUSER" value="450-CP153" x="-13" y="-106.5" size="1.778" layer="27" display="off"/>
 </element>
+<element name="U3" library="hardware" package="EMPTY" value="SCREW-M2X8" x="-14" y="-107.75"/>
+<element name="U4" library="hardware" package="EMPTY" value="SCREW-M2X8" x="-15" y="-109"/>
+<element name="U5" library="hardware" package="EMPTY" value="SCREW-M2X8" x="-16" y="-110.25"/>
+<element name="U6" library="hardware" package="EMPTY" value="SCREW-M2X8" x="-17" y="-111.5"/>
+<element name="U7" library="hardware" package="EMPTY" value="NUT-M2-SELFLOCK" x="-18" y="-112.75"/>
+<element name="U8" library="hardware" package="EMPTY" value="NUT-M2-SELFLOCK" x="-19" y="-114"/>
+<element name="U9" library="hardware" package="EMPTY" value="NUT-M2-SELFLOCK" x="-20" y="-115.25"/>
+<element name="U10" library="hardware" package="EMPTY" value="NUT-M2-SELFLOCK" x="-21" y="-116.5"/>
 </elements>
 <signals>
