File: a405-diode-distortion.sch (EAGLE design)
At the start: 54 parts, among them U1 FX2-20P-1.27DS, U2 FX2-20S-1.27DS

Commit message: A405 Update
Parts:
- removed O1: (no value), text:TITLE
- added U10, U7, U8, U9: NUT-M2-SELFLOCK, hardware:NUT-M2-SELFLOCK
- added U3, U4, U5, U6: SCREW-M2X8, hardware:SCREW-M2X8
- PCB1: value rev.A -> A405 rev.A
Other:
- moved on the sheet: U1, U2
Changed lines of the file:
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@@
 <?xml version="1.0" encoding="utf-8"?>
 <!DOCTYPE eagle SYSTEM "eagle.dtd">
-<eagle version="7.4.1">
+<eagle version="7.5.1">
 <drawing>
 <settings>
@@
 </classes>
 <parts>
-<part name="O1" library="text" deviceset="TITLE" device=""/>
-<part name="PCB1" library="module-footprints" deviceset="ST2-BOARD-50" device="" value="rev.A"/>
+<part name="PCB1" library="module-footprints" deviceset="ST2-BOARD-?" device="50" value="A405 rev.A"/>
 <part name="U1" library="hardware" deviceset="?" device="FX2-20P-1.27DS"/>
 <part name="U2" library="hardware" deviceset="?" device="FX2-20S-1.27DS"/>
@@
 <part name="O6" library="hardware" deviceset="450-C?" device="P157(15MM,WHITE/BLACK)"/>
 <part name="O7" library="hardware" deviceset="450-C?" device="P153(15MM,BLUE/WHITE)"/>
+<part name="U3" library="hardware" deviceset="*?" device="SCREW-M2X8"/>
+<part name="U4" library="hardware" deviceset="*?" device="SCREW-M2X8"/>
+<part name="U5" library="hardware" deviceset="*?" device="SCREW-M2X8"/>
+<part name="U6" library="hardware" deviceset="*?" device="SCREW-M2X8"/>
+<part name="U7" library="hardware" deviceset="*?" device="NUT-M2-SELFLOCK"/>
+<part name="U8" library="hardware" deviceset="*?" device="NUT-M2-SELFLOCK"/>
+<part name="U9" library="hardware" deviceset="*?" device="NUT-M2-SELFLOCK"/>
+<part name="U10" library="hardware" deviceset="*?" device="NUT-M2-SELFLOCK"/>
 </parts>
 <sheets>
@@
 </plain>
 <instances>
-<instance part="O1" gate="G$1" x="0" y="195.58"/>
-<instance part="PCB1" gate="G$1" x="111.76" y="198.12"/>
+<instance part="PCB1" gate="G$1" x="20.32" y="175.26"/>
 <instance part="PCB1" gate="G$6" x="12.7" y="152.4"/>
 <instance part="PCB1" gate="G$7" x="86.36" y="152.4"/>
 <instance part="PCB1" gate="G$8" x="12.7" y="121.92"/>
-<instance part="U1" gate="G$1" x="86.36" y="170.18"/>
-<instance part="U2" gate="G$1" x="86.36" y="162.56"/>
+<instance part="U1" gate="G$1" x="58.42" y="175.26"/>
+<instance part="U2" gate="G$1" x="86.36" y="175.26"/>
 <instance part="PWR1" gate="G$1" x="58.42" y="35.56" rot="R270"/>
 <instance part="PWR2" gate="G$1" x="58.42" y="0" rot="R270"/>
@@
 <instance part="O6" gate="G$1" x="274.32" y="-15.24"/>
 <instance part="O7" gate="G$1" x="231.14" y="-15.24"/>
+<instance part="U3" gate="G$1" x="48.26" y="167.64"/>
+<instance part="U4" gate="G$1" x="48.26" y="165.1"/>
+<instance part="U5" gate="G$1" x="76.2" y="167.64"/>
+<instance part="U6" gate="G$1" x="76.2" y="165.1"/>
+<instance part="U7" gate="G$1" x="48.26" y="162.56"/>
+<instance part="U8" gate="G$1" x="48.26" y="160.02"/>
+<instance part="U9" gate="G$1" x="76.2" y="162.56"/>
+<instance part="U10" gate="G$1" x="76.2" y="160.02"/>
 </instances>
 <busses>
@@
 </schematic>
 </drawing>
-<compatibility>
-<note version="6.3" minversion="6.2.2" severity="warning">
-Since Version 6.2.2 text objects can contain more than one line,
-which will not be processed correctly with this version.
-</note>
-</compatibility>
 </eagle>
