File: a406-4069-overdrive.brd (EAGLE design)
At the start: 100 x 50 mm, 75 parts, among them U1 FX2-20P-1.27DS, U10 NUT-M2-SELFLOCK, U2 FX2-20S-1.27DS, U3 SCREW-M2X8, U4 SCREW-M2X8, U5 SCREW-M2X8, U6 SCREW-M2X8, U7 NUT-M2-SELFLOCK, U8 NUT-M2-SELFLOCK, U9 NUT-M2-SELFLOCK

Commit message: A406 in T/H
Parts:
- C12, C13, C14, C15: value 22P -> 22P(TH); device capacitors:C-0805 -> capacitors:C050-024X044
- C5, C6, C7, C8, C9: value 100N -> 100N(TH); device capacitors:C-0805 -> capacitors:C050-024X044
- DA1, DA2: value NJM2068M -> NJM2068D; device ic-jrc:SO-8 -> ic-jrc:DIP-8
- L1, L2, L3: value BLM31AJ601SN1L -> BL01RN1A1F1J; device inductors:1206 -> inductors:BL01RN1A
- R10, R11, R12, R13, R16, R17, R18, R19, R2, R20, R21, R22, R23, R25, R26, R27, R28, R29, R3, R30, R6, R7: value 10K -> 10K(TH); device resistors:R-0805 -> resistors:R-0207/10
- R31, R32: value 15K -> 15K(TH); device resistors:R-0805 -> resistors:R-0207/10
- R33, R34, R4, R5, R8, R9: value 100K -> 100K(TH); device resistors:R-0805 -> resistors:R-0207/10
- moved U10 113.1 mm to (88.2, -101.8)
- moved U9 109.7 mm to (86.0, -101.8)
- moved U8 106.2 mm to (83.8, -101.8)
- moved U7 102.8 mm to (81.5, -101.8)
- moved U6 99.4 mm to (79.2, -101.8)
- moved U5 96.0 mm to (77.0, -101.8)
- moved U4 92.6 mm to (74.8, -101.8)
- moved U3 89.2 mm to (72.5, -101.8)
- moved O9 80.2 mm to (65.8, -101.8)
- moved O8 74.5 mm to (63.5, -101.8)
- moved O7 74.5 mm to (61.2, -101.8)
- moved O5 72.5 mm to (56.8, -101.8)
- moved O6 69.0 mm to (59.0, -101.8)
- moved O3 64.4 mm to (52.2, -101.8)
- moved O4 63.5 mm to (54.5, -101.8)
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Connections:
- net GND: now also R33.1, R34.1; no longer R33.2, R34.2
- net N$14: now also DA1.6; no longer DA1.2
- net N$17: now also DA1.7; no longer DA1.1
- net N$28: now also R33.2; no longer R33.1
- net N$31: now also DA1.2; no longer DA1.6
- net N$32: now also DA1.1; no longer DA1.7
- net N$37: now also R34.2; no longer R34.1
Routing:
- net N$15: track 23.5 -> 94.9 mm, vias 0 -> 1
- net N$20: track 38.2 -> 94.8 mm, vias 2 -> 0
- net N$31: track 9.30 -> 51.8 mm
- net N$30: track 23.7 -> 2.27 mm
- net N$61: track 44.8 -> 24.1 mm, vias 2 -> 0
- net N$14: track 10.6 -> 31.0 mm
- net N$17: track 43.4 -> 63.2 mm, vias 0 -> 1
- net N$39: track 31.7 -> 13.6 mm, vias 2 -> 0
- net N$65: track 23.1 -> 40.7 mm
- net N$26: track 19.0 -> 35.5 mm
- net N$35: track 9.30 -> 24.6 mm
- net N$64: track 9.30 -> 24.5 mm
- net N$18: track 4.60 -> 19.2 mm
- net N$5: track 9.30 -> 22.8 mm
- net N$1: track 18.7 -> 31.5 mm
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