File: d104-lofi-delay.brd (EAGLE design)
At the start: 100 x 50 mm, 99 parts, among them U1 SCREW-M2X8, U10 FX2-20S-1.27DS, U2 SCREW-M2X8, U3 NUT-M2-SELFLOCK, U4 NUT-M2-SELFLOCK, U5 FX2-20P-1.27DS, U6 SCREW-M2X8, U7 SCREW-M2X8, U8 NUT-M2-SELFLOCK, U9 NUT-M2-SELFLOCK

Commit message: D104 Knobs update
Parts:
- O4, O6: value 450-CP157(15MM,WHITE/BLACK) -> 450-CP153(15MM,BLUE/WHITE)
- R28, R29: value 100K -> NF
Changed lines of the file:
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@@
 <attribute name="MOUSER" value="450-CP155" x="-65" y="-14" size="1.778" layer="27" display="off"/>
 </element>
-<element name="O6" library="hardware" package="EMPTY" value="450-CP157(15MM,WHITE/BLACK)" x="-66" y="-15.25">
-<attribute name="MOUSER" value="450-CP157" x="-66" y="-15.25" size="1.778" layer="27" display="off"/>
+<element name="O6" library="hardware" package="EMPTY" value="450-CP153(15MM,BLUE/WHITE)" x="-66" y="-15.25">
+<attribute name="MOUSER" value="450-CP153" x="-66" y="-15.25" size="1.778" layer="27" display="off"/>
 </element>
-<element name="O4" library="hardware" package="EMPTY" value="450-CP157(15MM,WHITE/BLACK)" x="-67" y="-16.5">
-<attribute name="MOUSER" value="450-CP157" x="-67" y="-16.5" size="1.778" layer="27" display="off"/>
+<element name="O4" library="hardware" package="EMPTY" value="450-CP153(15MM,BLUE/WHITE)" x="-67" y="-16.5">
+<attribute name="MOUSER" value="450-CP153" x="-67" y="-16.5" size="1.778" layer="27" display="off"/>
 </element>
 <element name="U1" library="hardware" package="EMPTY" value="SCREW-M2X8" x="-68" y="-17.75"/>
@@
 <element name="U8" library="hardware" package="EMPTY" value="NUT-M2-SELFLOCK" x="-74" y="-25.25"/>
 <element name="U9" library="hardware" package="EMPTY" value="NUT-M2-SELFLOCK" x="-75" y="-26.5"/>
-<element name="R29" library="resistors" package="R-0805" value="100K" x="87.5" y="23" rot="R180">
-<attribute name="MOUSER" value="660-RK73H2ATTD1003F" x="87.5" y="23" size="1.778" layer="27" rot="R180" display="off"/>
-</element>
-<element name="R28" library="resistors" package="R-0805" value="100K" x="87.5" y="27" rot="R180">
-<attribute name="MOUSER" value="660-RK73H2ATTD1003F" x="87.5" y="27" size="1.778" layer="27" rot="R180" display="off"/>
-</element>
+<element name="R29" library="resistors" package="R-0805" value="NF" x="87.5" y="23" rot="R180"/>
+<element name="R28" library="resistors" package="R-0805" value="NF" x="87.5" y="27" rot="R180"/>
 </elements>
 <signals>
