File: d104-lofi-delay.sch (EAGLE design)
At the start: 99 parts, among them U1 SCREW-M2X8, U10 FX2-20S-1.27DS, U2 SCREW-M2X8, U3 NUT-M2-SELFLOCK, U4 NUT-M2-SELFLOCK, U5 FX2-20P-1.27DS, U6 SCREW-M2X8, U7 SCREW-M2X8, U8 NUT-M2-SELFLOCK, U9 NUT-M2-SELFLOCK

Commit message: D104 Knobs update
Parts:
- O4, O6: value 450-CP157(15MM,WHITE/BLACK) -> 450-CP153(15MM,BLUE/WHITE); device hardware:450-CP157(15MM,WHITE/BLACK) -> hardware:450-CP153(15MM,BLUE/WHITE)
- R28, R29: value 100K -> NF; device resistors:100K -> resistors:NF
Changed lines of the file:
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@@
 <part name="O3" library="hardware" deviceset="450-AA?" device="150(15MM,D,BLACK)"/>
 <part name="O2" library="hardware" deviceset="450-C?" device="P155(15MM,GRAY/WHITE)"/>
-<part name="O6" library="hardware" deviceset="450-C?" device="P157(15MM,WHITE/BLACK)"/>
-<part name="O4" library="hardware" deviceset="450-C?" device="P157(15MM,WHITE/BLACK)"/>
+<part name="O6" library="hardware" deviceset="450-C?" device="P153(15MM,BLUE/WHITE)" value="450-CP153(15MM,BLUE/WHITE)"/>
+<part name="O4" library="hardware" deviceset="450-C?" device="P153(15MM,BLUE/WHITE)" value="450-CP153(15MM,BLUE/WHITE)"/>
 <part name="U1" library="hardware" deviceset="*?" device="SCREW-M2X8"/>
 <part name="U2" library="hardware" deviceset="*?" device="SCREW-M2X8"/>
@@
 <part name="U8" library="hardware" deviceset="*?" device="NUT-M2-SELFLOCK"/>
 <part name="U9" library="hardware" deviceset="*?" device="NUT-M2-SELFLOCK"/>
-<part name="R29" library="resistors" deviceset="?" device="100K"/>
-<part name="R28" library="resistors" deviceset="?" device="100K"/>
+<part name="R29" library="resistors" deviceset="?" device="NF" value="NF"/>
+<part name="R28" library="resistors" deviceset="?" device="NF" value="NF"/>
 </parts>
 <sheets>
