File: m913-dev-adapter.brd (EAGLE design)
At the start: 100 x 26 mm, 23 parts, among them U1 SCREW-M2X8, U10 FX2-20S-1.27DS, U2 SCREW-M2X8, U3 NUT-M2-SELFLOCK, U4 NUT-M2-SELFLOCK, U5 FX2-20P-1.27DS, U6 SCREW-M2X8, U7 SCREW-M2X8, U8 NUT-M2-SELFLOCK, U9 NUT-M2-SELFLOCK

Commit message: Add CV knob
Parts:
- added O1: 450-AA150(15MM,D,BLACK), hardware:EMPTY
- added O2: 450-CP151(15MM,RED/WHITE), hardware:EMPTY
Changed lines of the file:
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@@
 </element>
 <element name="XP1" library="connectors" package="ML10" value="" x="88" y="13" rot="R90"/>
+<element name="O1" library="hardware" package="EMPTY" value="450-AA150(15MM,D,BLACK)" x="-8" y="-59.25">
+<attribute name="MOUSER" value="450-AA150" x="-8" y="-59.25" size="1.778" layer="27" display="off"/>
+</element>
+<element name="O2" library="hardware" package="EMPTY" value="450-CP151(15MM,RED/WHITE)" x="-9" y="-60.5"/>
 </elements>
 <signals>
