File: a314-q&d-vcf.sch (EAGLE design)
At the start: 39 parts, among them U1 SCREW-M2X8, U10 FX2-20S-1.27DS, U2 SCREW-M2X8, U3 NUT-M2-SELFLOCK, U4 NUT-M2-SELFLOCK, U5 FX2-20P-1.27DS, U6 SCREW-M2X8, U7 SCREW-M2X8, U8 NUT-M2-SELFLOCK, U9 NUT-M2-SELFLOCK

Commit message: A314 Prototyping in progress
Connections:
- new net N$19: C4.1, C5.2
- net GND: no longer C4.1
- net N$17: no longer C5.2
Other:
- moved on the sheet: C3, C4, C5, C8, DA2.1, R14, R6, R7
Changed lines of the file:
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@@
 <part name="C4" library="capacitors" deviceset="?" device="1N(FILM)"/>
 <part name="C5" library="capacitors" deviceset="?" device="1N(FILM)"/>
-<part name="GND7" library="supply" deviceset="GND" device=""/>
-<part name="GND8" library="supply" deviceset="GND" device=""/>
 <part name="R12" library="potentiometers" deviceset="2**?" device="A10K"/>
 <part name="C6" library="capacitors" deviceset="?" device="10N(FILM)"/>
@@
 <part name="R14" library="resistors" deviceset="?" device="100K(TH)"/>
 <part name="GND10" library="supply" deviceset="GND" device=""/>
+<part name="GND7" library="supply" deviceset="GND" device=""/>
 </parts>
 <sheets>
@@
 <instances>
 <instance part="PCB1" gate="G$1" x="20.32" y="-2.54"/>
-<instance part="PCB1" gate="G$2" x="109.22" y="-129.54"/>
+<instance part="PCB1" gate="G$2" x="109.22" y="-137.16"/>
 <instance part="PCB1" gate="G$3" x="38.1" y="-154.94"/>
-<instance part="PCB1" gate="G$4" x="223.52" y="-134.62"/>
+<instance part="PCB1" gate="G$4" x="223.52" y="-142.24"/>
 <instance part="PCB1" gate="G$5" x="38.1" y="-160.02" rot="R180"/>
 <instance part="PCB1" gate="G$6" x="12.7" y="-27.94"/>
@@
 <instance part="PWR3" gate="G$1" x="241.3" y="-27.94" rot="R270"/>
 <instance part="PWR4" gate="G$1" x="241.3" y="-48.26" rot="R270"/>
-<instance part="R6" gate="G$1" x="132.08" y="-137.16" rot="MR90"/>
-<instance part="GND3" gate="VR1" x="132.08" y="-152.4"/>
-<instance part="C3" gate="G$1" x="142.24" y="-137.16"/>
-<instance part="R7" gate="G$1" x="147.32" y="-144.78" rot="R90"/>
-<instance part="GND5" gate="VR1" x="147.32" y="-152.4"/>
+<instance part="R6" gate="G$1" x="132.08" y="-144.78" rot="MR90"/>
+<instance part="GND3" gate="VR1" x="132.08" y="-160.02"/>
+<instance part="C3" gate="G$1" x="142.24" y="-144.78"/>
+<instance part="R7" gate="G$1" x="147.32" y="-152.4" rot="R90"/>
+<instance part="GND5" gate="VR1" x="147.32" y="-160.02"/>
 <instance part="R8" gate="G$1" x="55.88" y="-86.36"/>
 <instance part="R9" gate="G$1" x="43.18" y="-86.36" rot="MR90"/>
 <instance part="GND6" gate="VR1" x="43.18" y="-96.52"/>
 <instance part="PWR1" gate="G$1" x="43.18" y="-78.74"/>
-<instance part="DA2" gate=".1" x="170.18" y="-134.62" rot="MR180"/>
+<instance part="DA2" gate=".1" x="170.18" y="-142.24" rot="MR180"/>
 <instance part="R10" gate="G$1" x="157.48" y="-111.76"/>
 <instance part="R11" gate="G$1" x="182.88" y="-111.76"/>
-<instance part="C4" gate="G$1" x="165.1" y="-116.84" rot="R90"/>
-<instance part="C5" gate="G$1" x="175.26" y="-116.84" rot="R90"/>
-<instance part="GND7" gate="VR1" x="165.1" y="-121.92"/>
-<instance part="GND8" gate="VR1" x="175.26" y="-121.92"/>
+<instance part="C4" gate="G$1" x="170.18" y="-116.84" rot="R90"/>
+<instance part="C5" gate="G$1" x="170.18" y="-124.46" rot="R90"/>
 <instance part="R12" gate=".1" x="182.88" y="-104.14" rot="MR0"/>
 <instance part="C6" gate="G$1" x="170.18" y="-104.14"/>
@@
 <instance part="HL1" gate="G$1" x="149.86" y="-93.98" rot="R270"/>
 <instance part="GND9" gate="VR1" x="149.86" y="-99.06"/>
-<instance part="C8" gate="G$1" x="195.58" y="-134.62"/>
-<instance part="R14" gate="G$1" x="200.66" y="-142.24" rot="R90"/>
-<instance part="GND10" gate="VR1" x="200.66" y="-152.4"/>
+<instance part="C8" gate="G$1" x="195.58" y="-142.24"/>
+<instance part="R14" gate="G$1" x="200.66" y="-149.86" rot="R90"/>
+<instance part="GND10" gate="VR1" x="200.66" y="-160.02"/>
+<instance part="GND7" gate="VR1" x="170.18" y="-129.54"/>
 </instances>
 <busses>
@@
 <pinref part="R6" gate="G$1" pin="CCW"/>
 <pinref part="GND3" gate="VR1" pin="GND"/>
-<wire x1="132.08" y1="-149.86" x2="132.08" y2="-142.24" width="0.1524" layer="91"/>
+<wire x1="132.08" y1="-157.48" x2="132.08" y2="-149.86" width="0.1524" layer="91"/>
 </segment>
 <segment>
@@
 </segment>
 <segment>
-<pinref part="C4" gate="G$1" pin="1"/>
-<pinref part="GND7" gate="VR1" pin="GND"/>
-</segment>
-<segment>
-<pinref part="C5" gate="G$1" pin="1"/>
-<pinref part="GND8" gate="VR1" pin="GND"/>
-</segment>
-<segment>
 <pinref part="HL1" gate="G$1" pin="C"/>
 <pinref part="GND9" gate="VR1" pin="GND"/>
@@
 <pinref part="GND10" gate="VR1" pin="GND"/>
 <pinref part="R14" gate="G$1" pin="1"/>
-<wire x1="200.66" y1="-149.86" x2="200.66" y2="-147.32" width="0.1524" layer="91"/>
+<wire x1="200.66" y1="-157.48" x2="200.66" y2="-154.94" width="0.1524" layer="91"/>
+</segment>
+<segment>
+<pinref part="C5" gate="G$1" pin="1"/>
+<pinref part="GND7" gate="VR1" pin="GND"/>
 </segment>
 </net>
@@
 <segment>
 <pinref part="PCB1" gate="G$2" pin="INL"/>
-<wire x1="129.54" y1="-129.54" x2="132.08" y2="-129.54" width="0.1524" layer="91"/>
+<wire x1="129.54" y1="-137.16" x2="132.08" y2="-137.16" width="0.1524" layer="91"/>
 <pinref part="R6" gate="G$1" pin="CW"/>
-<wire x1="132.08" y1="-129.54" x2="132.08" y2="-132.08" width="0.1524" layer="91"/>
+<wire x1="132.08" y1="-137.16" x2="132.08" y2="-139.7" width="0.1524" layer="91"/>
 </segment>
 </net>
@@
 <pinref part="R6" gate="G$1" pin="W"/>
 <pinref part="C3" gate="G$1" pin="1"/>
-<wire x1="137.16" y1="-137.16" x2="139.7" y2="-137.16" width="0.1524" layer="91"/>
+<wire x1="137.16" y1="-144.78" x2="139.7" y2="-144.78" width="0.1524" layer="91"/>
 </segment>
 </net>
@@
 <pinref part="C3" gate="G$1" pin="2"/>
 <pinref part="R7" gate="G$1" pin="2"/>
-<wire x1="144.78" y1="-137.16" x2="147.32" y2="-137.16" width="0.1524" layer="91"/>
-<wire x1="147.32" y1="-137.16" x2="147.32" y2="-139.7" width="0.1524" layer="91"/>
+<wire x1="144.78" y1="-144.78" x2="147.32" y2="-144.78" width="0.1524" layer="91"/>
+<wire x1="147.32" y1="-144.78" x2="147.32" y2="-147.32" width="0.1524" layer="91"/>
 <pinref part="DA2" gate=".1" pin="IN+"/>
-<wire x1="160.02" y1="-137.16" x2="147.32" y2="-137.16" width="0.1524" layer="91"/>
-<junction x="147.32" y="-137.16"/>
+<wire x1="160.02" y1="-144.78" x2="147.32" y2="-144.78" width="0.1524" layer="91"/>
+<junction x="147.32" y="-144.78"/>
 </segment>
 </net>
@@
 <segment>
 <pinref part="DA2" gate=".1" pin="IN-"/>
-<wire x1="160.02" y1="-132.08" x2="149.86" y2="-132.08" width="0.1524" layer="91"/>
-<wire x1="149.86" y1="-132.08" x2="149.86" y2="-111.76" width="0.1524" layer="91"/>
+<wire x1="160.02" y1="-139.7" x2="149.86" y2="-139.7" width="0.1524" layer="91"/>
+<wire x1="149.86" y1="-139.7" x2="149.86" y2="-111.76" width="0.1524" layer="91"/>
 <pinref part="R10" gate="G$1" pin="1"/>
 <wire x1="149.86" y1="-111.76" x2="152.4" y2="-111.76" width="0.1524" layer="91"/>
@@
 <pinref part="R10" gate="G$1" pin="2"/>
 <pinref part="R11" gate="G$1" pin="1"/>
-<wire x1="162.56" y1="-111.76" x2="165.1" y2="-111.76" width="0.1524" layer="91"/>
-<pinref part="C5" gate="G$1" pin="2"/>
-<wire x1="165.1" y1="-111.76" x2="175.26" y2="-111.76" width="0.1524" layer="91"/>
-<wire x1="175.26" y1="-111.76" x2="177.8" y2="-111.76" width="0.1524" layer="91"/>
-<wire x1="175.26" y1="-114.3" x2="175.26" y2="-111.76" width="0.1524" layer="91"/>
-<junction x="175.26" y="-111.76"/>
+<wire x1="162.56" y1="-111.76" x2="170.18" y2="-111.76" width="0.1524" layer="91"/>
+<wire x1="170.18" y1="-111.76" x2="177.8" y2="-111.76" width="0.1524" layer="91"/>
 <pinref part="C4" gate="G$1" pin="2"/>
-<wire x1="165.1" y1="-114.3" x2="165.1" y2="-111.76" width="0.1524" layer="91"/>
-<junction x="165.1" y="-111.76"/>
+<wire x1="170.18" y1="-114.3" x2="170.18" y2="-111.76" width="0.1524" layer="91"/>
+<junction x="170.18" y="-111.76"/>
 </segment>
 </net>
@@
 <pinref part="R11" gate="G$1" pin="2"/>
 <wire x1="187.96" y1="-111.76" x2="190.5" y2="-111.76" width="0.1524" layer="91"/>
-<wire x1="190.5" y1="-111.76" x2="190.5" y2="-134.62" width="0.1524" layer="91"/>
+<wire x1="190.5" y1="-111.76" x2="190.5" y2="-142.24" width="0.1524" layer="91"/>
 <pinref part="DA2" gate=".1" pin="OUT"/>
-<wire x1="190.5" y1="-134.62" x2="180.34" y2="-134.62" width="0.1524" layer="91"/>
+<wire x1="190.5" y1="-142.24" x2="180.34" y2="-142.24" width="0.1524" layer="91"/>
 <wire x1="190.5" y1="-111.76" x2="190.5" y2="-104.14" width="0.1524" layer="91"/>
 <junction x="190.5" y="-111.76"/>
@@
 <junction x="190.5" y="-104.14"/>
 <pinref part="C8" gate="G$1" pin="1"/>
-<wire x1="193.04" y1="-134.62" x2="190.5" y2="-134.62" width="0.1524" layer="91"/>
-<junction x="190.5" y="-134.62"/>
+<wire x1="193.04" y1="-142.24" x2="190.5" y2="-142.24" width="0.1524" layer="91"/>
+<junction x="190.5" y="-142.24"/>
 </segment>
 </net>
@@
 <segment>
 <pinref part="R14" gate="G$1" pin="2"/>
-<wire x1="200.66" y1="-137.16" x2="200.66" y2="-134.62" width="0.1524" layer="91"/>
+<wire x1="200.66" y1="-144.78" x2="200.66" y2="-142.24" width="0.1524" layer="91"/>
 <pinref part="C8" gate="G$1" pin="2"/>
-<wire x1="200.66" y1="-134.62" x2="198.12" y2="-134.62" width="0.1524" layer="91"/>
+<wire x1="200.66" y1="-142.24" x2="198.12" y2="-142.24" width="0.1524" layer="91"/>
 <pinref part="PCB1" gate="G$4" pin="OUTL"/>
-<wire x1="203.2" y1="-134.62" x2="200.66" y2="-134.62" width="0.1524" layer="91"/>
-<junction x="200.66" y="-134.62"/>
-</segment>
-</net>
+<wire x1="203.2" y1="-142.24" x2="200.66" y2="-142.24" width="0.1524" layer="91"/>
+<junction x="200.66" y="-142.24"/>
+</segment>
+</net>
+<net name="N$19" class="0">
+<segment>
+<pinref part="C5" gate="G$1" pin="2"/>
+<pinref part="C4" gate="G$1" pin="1"/>
+<wire x1="170.18" y1="-121.92" x2="170.18" y2="-119.38" width="0.1524" layer="91"/>
+</segment>
+</net>

Commit message: A314 Schematic and PCB
Parts:
- removed HL1: BLUE(3MM), optoelectronics:BLUE(3MM)
- added C10, C13, C14, C15, C16, C9: 100N(TH), capacitors:100N(TH)
- added C11, C12: 100N(FILM), capacitors:100N(FILM)
- added C17, C18: 22P(TH), capacitors:22P(TH)
- added DA3: NJM2068D, ic-jrc:NJM2068D
- added R15, R17, R18: 100K(TH), resistors:100K(TH)
- added R16: 2*B5K, potentiometers:2B5K
- added R19, R20, R21, R22: 10K(TH), resistors:10K(TH)
- added VT1, VT2: BC548, transistors-npn:BC548
- C3: value 100N(FILM) -> 47N(FILM); device capacitors:100N(FILM) -> capacitors:47N(FILM)
- C4: value 1N(FILM) -> 47N(FILM); device capacitors:1N(FILM) -> capacitors:47N(FILM)
- C5: value 1N(FILM) -> 22N(FILM); device capacitors:1N(FILM) -> capacitors:22N(FILM)
- C6: value 10N(FILM) -> 22N(FILM); device capacitors:10N(FILM) -> capacitors:22N(FILM)
- C7: value 10N(FILM) -> 10U/35V; device capacitors:10N(FILM) -> capacitors-electrolytic:10U/35V
- C8: value 100N(FILM) -> 10U/35V; device capacitors:100N(FILM) -> capacitors-electrolytic:10U/35V
- DA2: value NJM2068D -> TL072IP; device ic-jrc:NJM2068D -> ic-ti:TL072IP
- R1: value 100K(TH) -> B100K; device resistors:100K(TH) -> potentiometers:B100K
- R10: value 100K(TH) -> 68K(TH); device resistors:100K(TH) -> resistors:68K(TH)
- R12: value 2A10K -> 68K(TH); device potentiometers:2A10K -> resistors:68K(TH)
- R2: value B100K(CD)(9MM) -> 100K(TH); device potentiometers:B100K(CD)(9MM) -> resistors:100K(TH)
- R4: value 100K(TH) -> B100K(CD)(9MM); device resistors:100K(TH) -> potentiometers:B100K(CD)(9MM)
- R6: value 100K(64X/Z) -> 100K(TH); device potentiometers:100K(64X/Z) -> resistors:100K(TH)
- R9: value B100K -> 100K(TH); device potentiometers:B100K -> resistors:100K(TH)
Connections:
- new net N$21: C6.2, R16.2.CCW, R16.2.W
- new net N$22: C3.2, C5.1, R11.2, VT1.C
- new net N$26: C2.2, R12.1, VT2.B
- new net N$27: PCB1G$3.INR, R9.1
- new net N$28: DA1.2.OUT, R10.2, R12.2, R7.2
- new net N$29: C18.2, DA3.2.OUT, PCB1G$5.OUTR, R22.2
- new net N$30: C17.1, DA3.1.IN-, R19.2, R21.1
- new net N$31: C17.2, DA3.1.OUT, PCB1G$4.OUTL, R21.2
- net +15V: now also C13.2, C15.2, C7.+, C9.2, DA2*.V+, DA3*.V+, R1.CW; no longer C1.2, R9.CW
- net -15V: now also C10.1, C14.1, C16.1, C8.-, DA2*.V-, DA3*.V-; no longer C2.1
- net GND: now also C10.2, C13.1, C14.2, C15.1, C16.2, C2.1, C7.-, C8.+, C9.1, DA2.1.IN+, DA2.2.IN+, DA3.1.IN+, DA3.2.IN+, R1.CCW, R11.1, R13.1, R17.1, R18.1, VT1.E, VT2.E; no longer C2.2, C5.1, HL1.C, R14.1, R6.CCW, R7.1, R9.CCW
- net N$10: now also C4.1, DA2.2.IN-, R15.1, R9.2; no longer PCB1G$2.INL, R6.CW
- net N$11: now also DA2.1.IN-, R14.1, R8.2; no longer R6.W
- net N$12: now also PCB1G$2.INL, R8.1; no longer C3.2, DA2.1.IN+, R7.2
- net N$13: now also R1.W, R2.1; no longer R8.1, R9.W
- net N$14: now also C11.1, DA2.1.OUT, R14.2, R16.1.CW; no longer C7.1, DA2.1.IN-, R10.1
- net N$17: now also C11.2, R17.2, R19.1; no longer C4.2, R10.2, R11.1
- net N$18: now also C12.1, DA2.2.OUT, R15.2, R16.2.CW; no longer C8.1, DA2.1.OUT, R11.2, R12.1.CCW, R12.1.W
- net N$19: now also R16.1.CCW, R16.1.W; no longer C4.1
- net N$20: now also C12.2, R18.2, R20.1; no longer C6.2, R12.1.CW
- net N$23: now also C1.2, R10.1, VT1.B; no longer C6.1, C7.2, HL1.A, R13.2
- net N$24: now also C4.2, C6.1, R13.2, VT2.C; no longer C8.2, PCB1G$4.OUTL, R14.2
- net N$3: now also R3.2, R4.W; no longer R1.2, R2.W
- net N$5: now also R2.2, R4.CW, R5.1; no longer R2.CW, R3.1, R8.2
- net N$6: now also R5.2, R6.1; no longer R3.2, R4.1
- net N$7: now also R4.CCW, R6.2, R7.1; no longer R2.CCW, R4.2, R5.1
- net N$8: now also C18.1, DA3.2.IN-, R20.2, R22.1; no longer DA1.2.OUT, R13.1, R5.2
- net N$9: now also R3.1; no longer R1.1
Other:
- moved on the sheet: C1, C2, C3, C4, C5, C6, DA2.1, R10, R11, R13, R14, R3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

Commit message: A314 Add knobs
Parts:
- added O1, O2, O3: 450-AA150(15MM,D,BLACK), hardware:450-AA150(15MM,D,BLACK)
- added O4: 450-CP151(15MM,RED/WHITE), hardware:450-CP151(15MM,RED/WHITE)
- added O5, O6: 450-CP153(15MM,BLUE/WHITE), hardware:450-CP153(15MM,BLUE/WHITE)
- R16: value 2*B5K -> 2*A10K; device potentiometers:2B5K -> potentiometers:2A10K
Changed lines of the file:
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@@
 <part name="R17" library="resistors" deviceset="?" device="100K(TH)"/>
 <part name="GND9" library="supply" deviceset="GND" device=""/>
-<part name="R16" library="potentiometers" deviceset="2**?" device="B5K" value="2*B5K"/>
+<part name="R16" library="potentiometers" deviceset="2**?" device="A10K" value="2*A10K"/>
 <part name="C5" library="capacitors" deviceset="?" device="22N(FILM)"/>
 <part name="C3" library="capacitors" deviceset="?" device="47N(FILM)"/>
@@
 <part name="C7" library="capacitors-electrolytic" deviceset="?" device="10U/35V"/>
 <part name="C8" library="capacitors-electrolytic" deviceset="?" device="10U/35V"/>
+<part name="O1" library="hardware" deviceset="450-AA?" device="150(15MM,D,BLACK)"/>
+<part name="O2" library="hardware" deviceset="450-AA?" device="150(15MM,D,BLACK)"/>
+<part name="O3" library="hardware" deviceset="450-AA?" device="150(15MM,D,BLACK)"/>
+<part name="O4" library="hardware" deviceset="450-C?" device="P151(15MM,RED/WHITE)"/>
+<part name="O5" library="hardware" deviceset="450-C?" device="P153(15MM,BLUE/WHITE)"/>
+<part name="O6" library="hardware" deviceset="450-C?" device="P153(15MM,BLUE/WHITE)"/>
 </parts>
 <sheets>
@@
 <instance part="C7" gate="G$1" x="165.1" y="-33.02" rot="R270"/>
 <instance part="C8" gate="G$1" x="165.1" y="-43.18" rot="R270"/>
+<instance part="O1" gate="G$1" x="43.18" y="-111.76"/>
+<instance part="O2" gate="G$1" x="119.38" y="-60.96"/>
+<instance part="O3" gate="G$1" x="160.02" y="-101.6"/>
+<instance part="O4" gate="G$1" x="119.38" y="-60.96"/>
+<instance part="O5" gate="G$1" x="43.18" y="-111.76"/>
+<instance part="O6" gate="G$1" x="160.02" y="-101.6"/>
 </instances>
 <busses>

Commit message: A314 Add trimmer to set cutoff range
Parts:
- added R23: 10K(64W/Y), potentiometers:10K(64W/Y)
Connections:
- new net N$33: R1.CCW, R23.CW, R23.W
- net GND: now also R23.CCW; no longer R1.CCW
Changed lines of the file:
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@@
 <part name="O5" library="hardware" deviceset="450-C?" device="P153(15MM,BLUE/WHITE)"/>
 <part name="O6" library="hardware" deviceset="450-C?" device="P153(15MM,BLUE/WHITE)"/>
+<part name="R23" library="potentiometers" deviceset="?(64W/Y)" device="10K"/>
 </parts>
 <sheets>
@@
 <instance part="R2" gate="G$1" x="55.88" y="-86.36"/>
 <instance part="R1" gate="G$1" x="43.18" y="-86.36" rot="MR90"/>
-<instance part="GND1" gate="VR1" x="43.18" y="-96.52"/>
+<instance part="GND1" gate="VR1" x="43.18" y="-109.22"/>
 <instance part="PWR1" gate="G$1" x="43.18" y="-78.74"/>
 <instance part="DA2" gate=".1" x="154.94" y="-154.94" rot="MR180"/>
@@
 <instance part="C7" gate="G$1" x="165.1" y="-33.02" rot="R270"/>
 <instance part="C8" gate="G$1" x="165.1" y="-43.18" rot="R270"/>
-<instance part="O1" gate="G$1" x="43.18" y="-111.76"/>
+<instance part="O1" gate="G$1" x="43.18" y="-124.46"/>
 <instance part="O2" gate="G$1" x="119.38" y="-60.96"/>
 <instance part="O3" gate="G$1" x="160.02" y="-101.6"/>
 <instance part="O4" gate="G$1" x="119.38" y="-60.96"/>
-<instance part="O5" gate="G$1" x="43.18" y="-111.76"/>
+<instance part="O5" gate="G$1" x="43.18" y="-124.46"/>
 <instance part="O6" gate="G$1" x="160.02" y="-101.6"/>
+<instance part="R23" gate="G$1" x="43.18" y="-101.6" rot="R90"/>
 </instances>
 <busses>
@@
 </segment>
 <segment>
-<pinref part="R1" gate="G$1" pin="CCW"/>
 <pinref part="GND1" gate="VR1" pin="GND"/>
-<wire x1="43.18" y1="-91.44" x2="43.18" y2="-93.98" width="0.1524" layer="91"/>
+<pinref part="R23" gate="G$1" pin="CCW"/>
 </segment>
 <segment>
@@
 </segment>
 </net>
+<net name="N$33" class="0">
+<segment>
+<pinref part="R1" gate="G$1" pin="CCW"/>
+<wire x1="43.18" y1="-91.44" x2="43.18" y2="-93.98" width="0.1524" layer="91"/>
+<pinref part="R23" gate="G$1" pin="CW"/>
+<wire x1="43.18" y1="-93.98" x2="43.18" y2="-96.52" width="0.1524" layer="91"/>
+<pinref part="R23" gate="G$1" pin="W"/>
+<wire x1="38.1" y1="-101.6" x2="35.56" y2="-101.6" width="0.1524" layer="91"/>
+<wire x1="35.56" y1="-101.6" x2="35.56" y2="-93.98" width="0.1524" layer="91"/>
+<wire x1="35.56" y1="-93.98" x2="43.18" y2="-93.98" width="0.1524" layer="91"/>
+<junction x="43.18" y="-93.98"/>
+</segment>
+</net>
