File: a718-noise-source.sch (EAGLE design)
At the start: 38 parts, among them U1 SCREW-M2X8, U10 FX2-20S-1.27DS, U2 SCREW-M2X8, U3 NUT-M2-SELFLOCK, U4 NUT-M2-SELFLOCK, U5 FX2-20P-1.27DS, U6 SCREW-M2X8, U7 SCREW-M2X8, U8 NUT-M2-SELFLOCK, U9 NUT-M2-SELFLOCK

Commit message: A718 Update
Parts:
- added O1: 450-AA150(15MM,D,BLACK), hardware:450-AA150(15MM,D,BLACK)
- added O2: 450-CP156(15MM,BLACK/WHITE), hardware:450-CP156(15MM,BLACK/WHITE)
Changed lines of the file:
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@@
 <part name="R12" library="potentiometers" deviceset="?" device="A10K(9MM)"/>
 <part name="GND5" library="supply" deviceset="GND" device=""/>
+<part name="O1" library="hardware" deviceset="450-AA?" device="150(15MM,D,BLACK)"/>
+<part name="O2" library="hardware" deviceset="450-C?" device="P156(15MM,BLACK/WHITE)"/>
 </parts>
 <sheets>
@@
 <instance part="GND5" gate="VR1" x="170.18" y="-132.08"/>
 <instance part="DA1" gate="*" x="228.6" y="-45.72"/>
+<instance part="O1" gate="G$1" x="170.18" y="-144.78"/>
+<instance part="O2" gate="G$1" x="170.18" y="-144.78"/>
 </instances>
 <busses>

Commit message: A718 Fix Feedback
Parts:
- added R13, R14: 100K(TH), resistors:100K(TH)
Connections:
- net GND: now also R13.1, R14.1
- net N$17: now also PCB1G$6.RFBK
- net N$18: now also PCB1G$6.LFBK
- net N$3: now also R14.2; no longer PCB1G$6.RFBK
- net N$6: now also R13.2; no longer PCB1G$6.LFBK
Changed lines of the file:
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@@
 <part name="O1" library="hardware" deviceset="450-AA?" device="150(15MM,D,BLACK)"/>
 <part name="O2" library="hardware" deviceset="450-C?" device="P156(15MM,BLACK/WHITE)"/>
+<part name="R13" library="resistors" deviceset="?" device="100K(TH)"/>
+<part name="R14" library="resistors" deviceset="?" device="100K(TH)"/>
+<part name="GND7" library="supply" deviceset="GND" device=""/>
+<part name="GND8" library="supply" deviceset="GND" device=""/>
 </parts>
 <sheets>
@@
 <instance part="O1" gate="G$1" x="170.18" y="-144.78"/>
 <instance part="O2" gate="G$1" x="170.18" y="-144.78"/>
+<instance part="R13" gate="G$1" x="55.88" y="-66.04" rot="R90"/>
+<instance part="R14" gate="G$1" x="60.96" y="-66.04" rot="R90"/>
+<instance part="GND7" gate="VR1" x="55.88" y="-73.66"/>
+<instance part="GND8" gate="VR1" x="60.96" y="-73.66"/>
 </instances>
 <busses>
@@
 <wire x1="170.18" y1="-116.84" x2="170.18" y2="-129.54" width="0.1524" layer="91"/>
 </segment>
+<segment>
+<pinref part="R13" gate="G$1" pin="1"/>
+<pinref part="GND7" gate="VR1" pin="GND"/>
+</segment>
+<segment>
+<pinref part="R14" gate="G$1" pin="1"/>
+<pinref part="GND8" gate="VR1" pin="GND"/>
+</segment>
 </net>
 <net name="N$38" class="0">
@@
 <pinref part="PCB1" gate="G$6" pin="SENSE"/>
 <wire x1="66.04" y1="-58.42" x2="33.02" y2="-58.42" width="0.1524" layer="91"/>
-</segment>
-</net>
-<net name="N$3" class="0">
-<segment>
-<pinref part="PCB1" gate="G$6" pin="RFBK"/>
-<pinref part="PCB1" gate="G$7" pin="RFBK'"/>
-<wire x1="33.02" y1="-38.1" x2="66.04" y2="-38.1" width="0.1524" layer="91"/>
-</segment>
-</net>
-<net name="N$6" class="0">
-<segment>
-<pinref part="PCB1" gate="G$6" pin="LFBK"/>
-<pinref part="PCB1" gate="G$7" pin="LFBK'"/>
-<wire x1="33.02" y1="-35.56" x2="66.04" y2="-35.56" width="0.1524" layer="91"/>
 </segment>
 </net>
@@
 <pinref part="PCB1" gate="G$3" pin="INR"/>
 <pinref part="R4" gate="G$1" pin="2"/>
-<wire x1="33.02" y1="-20.32" x2="45.72" y2="-20.32" width="0.1524" layer="91"/>
+<wire x1="33.02" y1="-20.32" x2="40.64" y2="-20.32" width="0.1524" layer="91"/>
+<wire x1="40.64" y1="-20.32" x2="45.72" y2="-20.32" width="0.1524" layer="91"/>
 <wire x1="45.72" y1="-20.32" x2="45.72" y2="-22.86" width="0.1524" layer="91"/>
+<wire x1="40.64" y1="-20.32" x2="40.64" y2="-38.1" width="0.1524" layer="91"/>
+<junction x="40.64" y="-20.32"/>
+<pinref part="PCB1" gate="G$6" pin="RFBK"/>
+<wire x1="40.64" y1="-38.1" x2="33.02" y2="-38.1" width="0.1524" layer="91"/>
 </segment>
 </net>
@@
 <pinref part="PCB1" gate="G$2" pin="INL"/>
 <pinref part="R6" gate="G$1" pin="2"/>
-<wire x1="33.02" y1="-15.24" x2="50.8" y2="-15.24" width="0.1524" layer="91"/>
+<wire x1="33.02" y1="-15.24" x2="38.1" y2="-15.24" width="0.1524" layer="91"/>
+<wire x1="38.1" y1="-15.24" x2="50.8" y2="-15.24" width="0.1524" layer="91"/>
 <wire x1="50.8" y1="-15.24" x2="50.8" y2="-22.86" width="0.1524" layer="91"/>
+<wire x1="38.1" y1="-15.24" x2="38.1" y2="-35.56" width="0.1524" layer="91"/>
+<junction x="38.1" y="-15.24"/>
+<pinref part="PCB1" gate="G$6" pin="LFBK"/>
+<wire x1="38.1" y1="-35.56" x2="33.02" y2="-35.56" width="0.1524" layer="91"/>
 </segment>
 </net>
@@
 </segment>
 </net>
+<net name="N$3" class="0">
+<segment>
+<pinref part="R14" gate="G$1" pin="2"/>
+<wire x1="60.96" y1="-60.96" x2="60.96" y2="-38.1" width="0.1524" layer="91"/>
+<pinref part="PCB1" gate="G$7" pin="RFBK'"/>
+<wire x1="60.96" y1="-38.1" x2="66.04" y2="-38.1" width="0.1524" layer="91"/>
+</segment>
+</net>
+<net name="N$6" class="0">
+<segment>
+<pinref part="PCB1" gate="G$7" pin="LFBK'"/>
+<pinref part="R13" gate="G$1" pin="2"/>
+<wire x1="66.04" y1="-35.56" x2="55.88" y2="-35.56" width="0.1524" layer="91"/>
+<wire x1="55.88" y1="-35.56" x2="55.88" y2="-60.96" width="0.1524" layer="91"/>
+</segment>
+</net>
