File: a323-4pole-vcf.sch (EAGLE design)
At the start: 97 parts, among them U1 SCREW-M2X8, U10 FX2-20S-1.27DS, U2 SCREW-M2X8, U3 NUT-M2-SELFLOCK, U4 NUT-M2-SELFLOCK, U5 FX2-20P-1.27DS, U6 SCREW-M2X8, U7 SCREW-M2X8, U8 NUT-M2-SELFLOCK, U9 NUT-M2-SELFLOCK

Commit message: A323 TH Version
Parts:
- added C21: 100N(TH), capacitors:100N(TH)
- C1, C2, C28, C29: value 22P -> 22P(TH); device capacitors:22P -> capacitors:22P(TH)
- C10, C12, C13, C14, C15, C16, C17, C18, C19, C20, C9: value 100N -> 100N(TH); device capacitors:100N -> capacitors:100N(TH)
- DA1: value V2164M -> V2164D; device ic-coolaudio:V2164M -> ic-coolaudio:V2164D
- DA2: value TL074D -> TL074CN; device ic-ti:TL074D -> ic-ti:TL074CN
- DA3, DA6: value NJM2068M -> NJM2068D; device ic-jrc:NJM2068M -> ic-jrc:NJM2068D
- DA4, DA5: value TL072ID -> TL072IP; device ic-ti:TL072ID -> ic-ti:TL072IP
- L1, L2: value BLM31AJ601SN1L -> BL01RN1A1F1J; device inductors:BLM31AJ601SN1L -> inductors:BL01RN1A1F1J
- PCB1: device module-footprints:ST2-BOARD-50 -> module-footprints:ST2-BOARD-74
- R10, R12, R13, R17, R18, R19, R20, R22, R24, R36, R37, R40, R41, R9: value 10K -> 10K(TH); device resistors:10K -> resistors:10K(TH)
- R14, R15, R6, R7: value 4K7 -> 4K7(TH); device resistors:4K7 -> resistors:4K7(TH)
- R16, R2, R3, R5, R8: value 100K -> 100K(TH); device resistors:100K -> resistors:100K(TH)
- R21, R25: value 20K -> 20K(TH); device resistors:20K -> resistors:20K(TH)
- R23: value 18K -> 18K(TH); device resistors:18K -> resistors:18K(TH)
- R26, R27, R28, R29: value 30K -> 30K(TH); device resistors:30K -> resistors:30K(TH)
- R30, R31, R32, R33: value 470R -> 470R(TH); device resistors:470R -> resistors:470R(TH)
- R34: value 39K -> 39K(TH); device resistors:39K -> resistors:39K(TH)
- R35: value 2K7 -> 2K7(TH); device resistors:2K7 -> resistors:2K7(TH)
- R38, R39: value 12K -> 12K(TH); device resistors:12K -> resistors:12K(TH)
- VD1: value BAS16 -> BAT46; device diodes:BAS16 -> diodes-schottky:BAT46
Connections:
- net -15V: now also C21.1
- net GND: now also C21.2
- net N$19: now also SA2.1.3; no longer SA2.2.3
- net N$32: now also SA2.1.CM; no longer SA2.2.CM
- net N$33: now also SA2.2.3; no longer SA2.1.3
- net N$35: now also SA2.1.2; no longer SA2.2.2
- net N$37: now also SA2.1.1; no longer SA2.2.1
- net N$40: now also SA2.2.1; no longer SA2.1.1
- net N$44: now also SA2.2.2; no longer SA2.1.2
- net N$49: now also SA2.2.CM; no longer SA2.1.CM
Other:
- moved on the sheet: SA2.1, SA2.2

Commit message: A323 Opamps update
Parts:
- DA4, DA5: value TL072IP -> NJM2068D; device ic-ti:TL072IP -> ic-jrc:NJM2068D
Changed lines of the file:
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@@
 <part name="GND4" library="supply" deviceset="GND" device=""/>
 <part name="GND7" library="supply" deviceset="GND" device=""/>
-<part name="DA4" library="ic-ti" deviceset="TL072" device="IP" value="TL072IP"/>
-<part name="DA5" library="ic-ti" deviceset="TL072" device="IP" value="TL072IP"/>
+<part name="DA4" library="ic-jrc" deviceset="NJM2068" device="D" value="NJM2068D"/>
+<part name="DA5" library="ic-jrc" deviceset="NJM2068" device="D" value="NJM2068D"/>
 <part name="C22" library="capacitors" deviceset="?" device="1N(FILM)"/>
 <part name="C23" library="capacitors" deviceset="?" device="1N(FILM)"/>

Commit message: A323 Update to LM13700
Parts:
- removed C27: 10U/35V, capacitors-electrolytic:10U/35V
- removed C28, C29: 22P(TH), capacitors:22P(TH)
- added DA7: NJM13700D, ic-jrc:NJM13700D
- added R42, R43, R46, R47: 4K7(TH), resistors:4K7(TH)
- added R44, R45: 3K3(TH), resistors:3K3(TH)
- added VT1, VT3: BC548, transistors-npn:BC548
- added VT2: BC558, transistors-pnp:BC558
- C11, C7, C8: value 10U/35V -> 100N(TH); device capacitors-electrolytic:10U/35V -> capacitors:100N(TH)
- C13, C14, C21: value 100N(TH) -> 4N7(FILM); device capacitors:100N(TH) -> capacitors:4N7(FILM)
- C22: value 1N(FILM) -> 4N7(FILM); device capacitors:1N(FILM) -> capacitors:4N7(FILM)
- C23, C24: value 1N(FILM) -> 10U/35V; device capacitors:1N(FILM) -> capacitors-electrolytic:10U/35V
- C25: value 1N(FILM) -> 22P(TH); device capacitors:1N(FILM) -> capacitors:22P(TH)
- C26: value 10U/35V -> 22P(TH); device capacitors-electrolytic:10U/35V -> capacitors:22P(TH)
- C3, C4: value 470P(FILM) -> 10U/35V; device capacitors:470P(FILM) -> capacitors-electrolytic:10U/35V
- C5, C6: value 470P(FILM) -> 100N(TH); device capacitors:470P(FILM) -> capacitors:100N(TH)
- DA1: value V2164D -> TL074CN; device ic-coolaudio:V2164D -> ic-ti:TL074CN
- DA2: value TL074CN -> NJM2068D; device ic-ti:TL074CN -> ic-jrc:NJM2068D
- DA6: value NJM2068D -> NJM13700D; device ic-jrc:NJM2068D -> ic-jrc:NJM13700D
- R11: value 2B50K -> 10K(TH); device potentiometers:2B50K -> resistors:10K(TH)
- R12: value 10K(TH) -> 1K(TH); device resistors:10K(TH) -> resistors:1K(TH)
- R13: value 10K(TH) -> 100K(TH); device resistors:10K(TH) -> resistors:100K(TH)
- R14, R15, R7: value 4K7(TH) -> 100K(TH); device resistors:4K7(TH) -> resistors:100K(TH)
- R16: value 100K(TH) -> 30K(TH); device resistors:100K(TH) -> resistors:30K(TH)
- R2: value 100K(TH) -> 220K(TH); device resistors:100K(TH) -> resistors:220K(TH)
- R20: value 10K(TH) -> 6K8(TH); device resistors:10K(TH) -> resistors:6K8(TH)
- R21, R25: value 20K(TH) -> 10K(TH); device resistors:20K(TH) -> resistors:10K(TH)
- R23: value 18K(TH) -> 10K(TH); device resistors:18K(TH) -> resistors:10K(TH)
- R26: value 30K(TH) -> 10K(TH); device resistors:30K(TH) -> resistors:10K(TH)
- R27: value 30K(TH) -> 2A10K; device resistors:30K(TH) -> potentiometers:2A10K
- R28, R29: value 30K(TH) -> 3K3(TH); device resistors:30K(TH) -> resistors:3K3(TH)
- R3: value 100K(TH) -> 1M2(TH); device resistors:100K(TH) -> resistors:1M2(TH)
- R30, R31: value 470R(TH) -> 4K7(TH); device resistors:470R(TH) -> resistors:4K7(TH)
- R32, R33: value 470R(TH) -> 180R(TH); device resistors:470R(TH) -> resistors:180R(TH)
- R34: value 39K(TH) -> 180R(TH); device resistors:39K(TH) -> resistors:180R(TH)
- R35: value 2K7(TH) -> 180R(TH); device resistors:2K7(TH) -> resistors:180R(TH)
- R36, R37: value 10K(TH) -> 4K7(TH); device resistors:10K(TH) -> resistors:4K7(TH)
- R38, R39: value 12K(TH) -> 180R(TH); device resistors:12K(TH) -> resistors:180R(TH)
- R4: value B100K(CD)(9MM) -> 100K(TH); device potentiometers:B100K(CD)(9MM) -> resistors:100K(TH)
- R40, R41: value 10K(TH) -> 180R(TH); device resistors:10K(TH) -> resistors:180R(TH)
- R6: value 4K7(TH) -> B100K(CD)(9MM); device resistors:4K7(TH) -> potentiometers:B100K(CD)(9MM)
- R9: value 10K(TH) -> 3K9(TH); device resistors:10K(TH) -> resistors:3K9(TH)
- VD1: value BAT46 -> 1N4148; device diodes-schottky:BAT46 -> diodes:1N4148
Connections:
- new net FREQ_DC: DA6.1.AMP_BIAS, DA6.2.AMP_BIAS, DA7.1.AMP_BIAS, DA7.2.AMP_BIAS, R9.1
- new net N$58: PCB1G$3.INR, R11.1
- new net N$59: DA1.1.IN-, DA1.1.OUT
- net +15V: now also C11.2, C15.2, C17.2, C19.2, C3.+, C5.2, C7.2, DA7*.V+, R1.CW; no longer C12.2, C14.2, C16.2, C18.2, C20.2, C7.+
- net -15V: now also C12.1, C16.1, C18.1, C20.1, C4.-, C6.1, C8.1, DA7*.V-, R3.1; no longer C13.1, C15.1, C17.1, C19.1, C21.1, C8.-, R1.CW, R34.1
- net GND: now also C11.1, C12.2, C15.1, C16.2, C17.1, C18.2, C19.1, C20.2, C3.-, C4.+, C6.2, C7.1, C8.2, DA1.1.IN+, DA1.2.IN+, DA1.3.IN+, DA3.1.IN+, DA3.2.IN+, R12.1, R13.1, R17.1, R18.1, R2.1, R20.1, R28.1, R29.1, R32.1, R33.1, R34.1, R35.1, R38.1, R39.1, R40.1, R41.1, R44.1, R45.1, VD1.C, VT1.B, VT1.C, VT3.C; no longer C11.-, C12.1, C13.2, C14.1, C15.2, C16.1, C17.2, C18.1, C19.2, C20.1, C21.2, C3.1, C4.1, C6.1, C7.-, C8.+, DA2.2.IN+, DA2.3.IN+, DA2.4.IN+, DA6.1.IN+, DA6.2.IN+, R15.1, R22.1, R24.1, R38.2, R39.2, R6.2, R7.2
- net N$10: now also R12.2, R16.1, VT3.B; no longer C1.1, DA3.1.IN-, R17.2, R18.2, R9.2
- net N$11: now also R42.1, SA2.1.CM; no longer DA3.1.IN+, R10.2, R14.2
- net N$12: now also C1.1, DA2.1.IN-, R10.2, R13.2, R21.1, R22.1; no longer R10.1, R11.1.W
- net N$13: now also R4.1; no longer R2.1
- net N$14: now also DA1.4.IN-, VD1.A, VT2.E, VT3.E; no longer R11.1.CCW, R6.1
- net N$17: now also DA1.4.OUT, VT2.B; no longer R21.1, R22.2, R23.1
- net N$18: now also R9.2, VT2.C; no longer DA1.1.IN1, R26.2, R30.2
- net N$19: now also DA1.4.IN+, R2.2, R3.2, VT1.E; no longer C1.2, DA3.1.OUT, R17.1, R27.1, SA2.1.3
- net N$20: now also DA2.1.IN+, R17.2, R23.1; no longer DA1.1.IN2, R27.2, R31.2
- net N$21: now also R23.2, R27.1.W; no longer DA1.1.IN3, R28.2, R32.2
- net N$22: now also R27.1.CCW, R28.2; no longer DA1.1.IN4, R29.2, R33.2
- net N$23: now also C1.2, DA2.1.OUT, R22.2, SA2.1.3; no longer C3.2
- net N$24: now also DA6.2.IN+, R30.2, R34.2; no longer C4.2, R31.1
- net N$26: now also DA6.2.IN-, R32.2; no longer C5.2, R32.1
- net N$27: now also C13.1, DA4.2.IN-, DA6.2.OUT; no longer C6.2, R33.1
- net N$28: now also DA1.3.OUT, R15.2, R19.2; no longer DA2.3.OUT, R16.2, R21.2
- net N$29: now also C13.2, DA4.2.OUT, R27.1.CW, R36.1, SA2.1.2; no longer DA3.2.IN+, R13.2, R15.2
- net N$3: now also R5.2, R6.W; no longer R3.2, R4.W
- net N$30: now also DA7.2.IN+, R36.2, R40.2; no longer R11.2.W, R13.1
- net N$31: now also DA7.2.IN-, R38.2; no longer R11.2.CCW, R7.1
- net N$32: now also C23.-, R42.2; no longer C26.+, SA2.1.CM
- net N$33: now also C21.1, DA5.2.IN-, DA7.2.OUT; no longer C2.2, DA3.2.OUT, R19.1, R28.1, SA2.2.3
- net N$34: now also C21.2, DA5.2.OUT, R21.2, SA2.1.1; no longer C22.1, DA1.1.OUT2, DA4.1.IN-
- net N$35: now also C23.+, C25.1, DA3.1.IN-, R44.2, R46.1; no longer C22.2, DA4.1.OUT, R11.1.CW, R26.1, SA2.1.2
- net N$36: now also C25.2, DA3.1.OUT, PCB1G$4.OUTL, R46.2; no longer C23.1, DA1.1.OUT1, DA5.1.IN-
- net N$37: now also C2.1, DA2.2.IN-, R11.2, R14.2, R24.1, R25.1; no longer C23.2, DA5.1.OUT, R18.1, SA2.1.1
- net N$39: now also DA2.2.IN+, R18.2, R26.1; no longer C24.1, DA1.1.OUT4, DA5.2.IN-
- net N$40: now also R26.2, R27.2.W; no longer C24.2, DA5.2.OUT, R20.1, SA2.2.1
- net N$41: now also R27.2.CCW, R29.2; no longer C25.1, DA1.1.OUT3, DA4.2.IN-
- net N$44: now also C2.2, DA2.2.OUT, R25.2, R31.1, SA2.2.3; no longer C25.2, DA4.2.OUT, R11.2.CW, R29.1, SA2.2.2
- net N$45: now also DA6.1.IN+, R31.2, R35.2; no longer C26.-, R36.2
- net N$46: now also R33.2; no longer C28.1, R36.1, R38.1, R40.2
- net N$47: now also C14.1, DA4.1.IN-, DA6.1.OUT; no longer PCB1G$2.INL, R9.1
- net N$48: now also C14.2, DA4.1.OUT, R27.2.CW, R37.1, SA2.2.2; no longer C28.2, DA6.1.OUT, PCB1G$4.OUTL, R40.1
- net N$49: now also DA7.1.IN+, R37.2, R41.2; no longer C27.+, SA2.2.CM
- net N$5: now also DA1.2.IN-, R4.2, R6.CW, R7.1; no longer DA2.2.IN-, R2.2, R4.CCW, R5.1
- net N$50: now also DA7.1.IN-, R39.2; no longer C27.-, R37.2
- net N$51: now also C22.1, DA5.1.IN-, DA7.1.OUT; no longer C29.1, DA6.2.IN-, R37.1, R39.1, R41.2
- net N$52: now also C22.2, DA5.1.OUT, R24.2, SA2.2.1; no longer C29.2, DA6.2.OUT, PCB1G$5.OUTR, R41.1
- net N$53: now also R43.1, SA2.2.CM; no longer DA2.1.OUT, VD1.C
- net N$54: now also C24.-, R43.2; no longer DA2.1.IN+, DA2.4.OUT, R25.2, R35.2
- net N$55: now also C24.+, C26.1, DA3.2.IN-, R45.2, R47.1; no longer DA2.1.IN-, DA2.4.IN-, R23.2, R24.2, R25.1, VD1.A
- net N$56: now also C26.2, DA3.2.OUT, PCB1G$5.OUTR, R47.2; no longer PCB1G$3.INR, R12.1
- net N$57: now also PCB1G$2.INL, R10.1; no longer C11.+, DA1.1.CV1, DA1.1.CV2, DA1.1.CV3, DA1.1.CV4, R34.2, R35.1
- net N$6: now also DA1.2.OUT, R7.2; no longer DA2.2.OUT, R5.2
- net N$7: now also DA1.3.IN-, R15.1, R6.CCW; no longer DA2.3.IN-, R16.1, R4.CW
- net N$8: now also R16.2, R19.1; no longer C2.1, DA3.2.IN-, R12.2, R19.2
- net N$9: now also R5.1; no longer R3.1
Other:
- moved on the sheet: C1, C10, C12, C13, C14, C15, C16, C17, C18, C19, C2, C20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
