File: a124-vca.brd (EAGLE design)
At the start: 100 x 74 mm, 112 parts, among them U1 SCREW-M2X8, U10 FX2-20S-1.27DS, U2 SCREW-M2X8, U3 NUT-M2-SELFLOCK, U4 NUT-M2-SELFLOCK, U5 FX2-20P-1.27DS, U6 SCREW-M2X8, U7 SCREW-M2X8, U8 NUT-M2-SELFLOCK, U9 NUT-M2-SELFLOCK

Commit message: A124 Update
Parts:
- PCB1: value A323 rev.A -> A124 rev.A
Changed lines of the file:
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@@
 </autorouter>
 <elements>
-<element name="PCB1" library="module-footprints" package="ST2-BOARD-74" value="A323 rev.A" x="0" y="0"/>
+<element name="PCB1" library="module-footprints" package="ST2-BOARD-74" value="A124 rev.A" x="0" y="0"/>
 <element name="U5" library="hardware" package="EMPTY" value="FX2-20P-1.27DS" x="62" y="-142">
 <attribute name="MOUSER" value="798-FX2-20P-1.27DS71" x="0" y="-86" size="1.778" layer="27" display="off"/>
