File: a323-vcf.brd (EAGLE design)
At the start: 100 x 74 mm, 105 parts, among them U1 SCREW-M2X8, U10 FX2-20S-1.27DS, U2 SCREW-M2X8, U3 NUT-M2-SELFLOCK, U4 NUT-M2-SELFLOCK, U5 FX2-20P-1.27DS, U6 SCREW-M2X8, U7 SCREW-M2X8, U8 NUT-M2-SELFLOCK, U9 NUT-M2-SELFLOCK

Commit message: BC558 -> BC556 Update
Parts:
- VT2: value BC558 -> BC556
Changed lines of the file:
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@@
 </element>
 <element name="VT3" library="transistors-npn" package="TO92" value="BC548" x="11" y="52" rot="R180"/>
-<element name="VT2" library="transistors-pnp" package="TO92" value="BC558" x="11" y="46"/>
+<element name="VT2" library="transistors-pnp" package="TO92" value="BC556" x="11" y="46"/>
 <element name="R9" library="resistors" package="R-0207/10" value="3K9(TH)" x="17" y="49" rot="R90"/>
 <element name="VD1" library="diodes" package="DO35-7" value="1N4148" x="15" y="49" rot="R90">
