File: m303-stereo-output.sch (EAGLE design)
At the start: 76 parts, among them U1 SCREW-M2X8, U2 SCREW-M2X8, U3 NUT-M2-SELFLOCK, U4 NUT-M2-SELFLOCK, U5 FX2-20S-1.27DS, U6 ERM1-5MM

Commit message: M303 rev.D: Updated signal indicator
Parts:
- added R31: 1K(TH), resistors:1K(TH)
- added R32: 300K(TH), resistors:300K(TH)
- DA4: value LM2903N -> TL072IP; device ic-fairchild:LM2903N -> ic-ti:TL072IP
- HL1: value RED/BLUE(2MMX5MM,CC) -> RED/GREEN(2MMX5MM,CC); device optoelectronics:RED/BLUE(2MMX5MM,CC) -> optoelectronics:RED/GREEN(2MMX5MM,CC)
- PCB1: value M303 rev.C -> M303 rev.D
- R18, R20: value 10M(TH) -> 1M(TH); device resistors:10M(TH) -> resistors:1M(TH)
- R19, R21: value 100K(TH) -> 33K(TH); device resistors:100K(TH) -> resistors:33K(TH)
- R25: value 22K(TH) -> 10K(TH); device resistors:22K(TH) -> resistors:10K(TH)
- R26: value 4K7(TH) -> 470K(TH); device resistors:4K7(TH) -> resistors:470K(TH)
- R27: value 100R(TH) -> 15K(TH); device resistors:100R(TH) -> resistors:15K(TH)
- R28: value 10K(TH) -> 100K(TH); device resistors:10K(TH) -> resistors:100K(TH)
- R29: value 2K2(TH) -> 100K(TH); device resistors:2K2(TH) -> resistors:100K(TH)
- R30: value 1K8(TH) -> 1K(TH); device resistors:1K8(TH) -> resistors:1K(TH)
Connections:
- removed net N$23 (its old number): DA4.1.IN-, R26.1, R27.2
- removed net N$25: DA4.1.OUT, HL1.A2, R30.1, VT1.C
- removed net N$47: DA4.2.IN-, R25.1, R26.2
- removed net N$48: DA4.2.OUT, HL1.A1, R28.2, R29.1
- removed net N$49: R28.1, VT1.B
- new net N$13: DA4.2.IN-, R25.2, R28.1
- new net N$17: DA4.2.OUT, R28.2, R30.1
- new net N$29: HL1.A2, R30.2, VT1.C
- new net N$30: DA4.1.IN-, R26.2, R27.2, R29.1
- new net N$31: DA4.1.OUT, R29.2, R31.1, R32.1
- new net N$32: R32.2, VT1.B
- new net N$33: HL1.A1, R31.2
- net +15V: now also R26.1; no longer R25.2
- net -15V: no longer HL1.K, VT1.E
- net GND: now also HL1.K, R25.1, VT1.E; no longer R29.2, R30.2
Other:
- moved on the sheet: DA4.1, DA4.2, HL1, R25, R26, R27, R28, R29, R30, U6, VT1

Commit message: M303d Resistor Value Update
Parts:
- R32: value 300K(TH) -> 330K(TH); device resistors:300K(TH) -> resistors:330K(TH)
Changed lines of the file:
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@@
 <part name="R27" library="resistors" deviceset="?" device="15K(TH)"/>
 <part name="R26" library="resistors" deviceset="?" device="470K(TH)"/>
-<part name="R32" library="resistors" deviceset="?" device="300K(TH)"/>
+<part name="R32" library="resistors" deviceset="?" device="330K(TH)" value="330K(TH)"/>
 <part name="R31" library="resistors" deviceset="?" device="1K(TH)"/>
 <part name="R30" library="resistors" deviceset="?" device="1K(TH)"/>
