File: m202-stereo-input.brd (EAGLE design)
At the start: 100 x 50 mm, 77 parts, among them U1 SCREW-M2X8, U10 FX2-20S-1.27DS, U11 ERM1-5MM, U2 SCREW-M2X8, U3 NUT-M2-SELFLOCK, U4 NUT-M2-SELFLOCK, U5 FX2-20P-1.27DS, U6 SCREW-M2X8, U7 SCREW-M2X8, U8 NUT-M2-SELFLOCK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

Commit message: M202d: Improved signal indicator
Parts:
- added R32: 1K(TH), resistors:R-0207/10
- added R33: 300K(TH), resistors:R-0207/10
- DA3: value LM2903N -> TL072IP; device ic-fairchild:DIP-8 -> ic-ti:DIP-8
- HL1: value RED/BLUE(2MMX5MM,CC) -> RED/GREEN(2MMX5MM,CC)
- PCB1: value M202 rev.C -> M202 rev.D
- R24: value 22K(TH) -> 10K(TH)
- R25: value 4K7(TH) -> 470K(TH)
- R26: value 100R(TH) -> 15K(TH)
- R29: value 10K(TH) -> 100K(TH)
- R30: value 2K2(TH) -> 100K(TH)
- R31: value 1K8(TH) -> 1K(TH)
- moved U11 89.3 mm to (7.00, -138.0)
- moved R25 11.4 mm to (27.0, 32.5), turned to 180 degrees
- moved R29 11.0 mm to (22.0, 45.0), turned to 180 degrees
- moved R16 9.06 mm to (36.0, 32.0), turned to 90 degrees
- moved VD2 8.06 mm to (42.0, 31.0), turned to 0 degrees
- moved R24 7.43 mm to (29.0, 40.0), turned to 90 degrees
- moved R6 7.28 mm to (51.0, 29.0), turned to 90 degrees
- moved R17 7.07 mm to (34.0, 32.0), turned to 90 degrees
- moved R3 6.40 mm to (49.0, 29.0), turned to 90 degrees
- moved VD1 5.70 mm to (42.0, 33.5), turned to 0 degrees
- moved C9 5.59 mm to (16.0, 39.0), turned to 90 degrees
- moved R30 3.35 mm to (14.0, 40.0)
- moved C6 3.16 mm to (50.0, 20.0), turned to 90 degrees
- moved C10 1.00 mm to (35.0, 39.0)
- moved C17 1.00 mm to (35.0, 42.0)
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Connections:
- removed net N$46: DA3.2, R25.1, R26.2
- removed net N$47: DA3.6, R24.1, R25.2
- removed net N$48: DA3.7, HL1.A1, R29.2, R30.1
- removed net N$49: R29.1, VT1.2
- removed net N$51: DA3.1, HL1.A2, R31.1, VT1.1
- new net N$18: DA3.6, R24.2, R29.1
- new net N$20: DA3.7, R29.2, R31.1
- new net N$21: HL1.A2, R31.2, VT1.1
- new net N$22: DA3.2, R25.2, R26.2, R30.1
- new net N$23: DA3.1, R30.2, R32.1, R33.1
- new net N$25: R33.2, VT1.2
- new net N$33: HL1.A1, R32.2
- net +15V: now also R25.1; no longer R24.2
- net -15V: no longer HL1.K, VT1.3
- net GND: now also HL1.K, R24.1, VT1.3; no longer R30.2, R31.2
Routing:
- net N$20: track 0.00 -> 31.5 mm
- net N$22: track 0.00 -> 25.2 mm
- net -15V: track 128.4 -> 104.3 mm
- net N$48: track 22.5 -> 0.00 mm
- net N$51: track 20.8 -> 0.00 mm
- net N$47: track 14.0 -> 0.00 mm
- net N$21: track 0.00 -> 11.2 mm
- net N$33: track 0.00 -> 10.7 mm
- net N$44: track 3.61 -> 14.1 mm
- net N$23: track 0.00 -> 9.95 mm
- net N$45: track 24.6 -> 34.4 mm
- net N$46: track 9.78 -> 0.00 mm
- net N$25: track 0.00 -> 9.68 mm
- net N$17: track 16.9 -> 24.4 mm
- net N$31: track 9.24 -> 15.7 mm
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
Commit message: M202d: Resistor values fix
Parts:
- R12, R14: value 10M(TH) -> 1M(TH)
- R13, R15: value 100K(TH) -> 33K(TH)
Changed lines of the file:
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@@
 <attribute name="NAME" x="22.095" y="25" size="0.8128" layer="25" ratio="15" rot="R90" align="center"/>
 </element>
-<element name="R12" library="resistors" package="R-0207/10" value="10M(TH)" x="16.5" y="25" smashed="yes" rot="R270">
+<element name="R12" library="resistors" package="R-0207/10" value="1M(TH)" x="16.5" y="25" smashed="yes" rot="R270">
 <attribute name="NAME" x="16.5" y="25" size="0.8128" layer="25" ratio="15" rot="R270" align="center"/>
 </element>
-<element name="R14" library="resistors" package="R-0207/10" value="10M(TH)" x="20.5" y="25" smashed="yes" rot="R270">
+<element name="R14" library="resistors" package="R-0207/10" value="1M(TH)" x="20.5" y="25" smashed="yes" rot="R270">
 <attribute name="NAME" x="20.5" y="25" size="0.8128" layer="25" ratio="15" rot="R270" align="center"/>
 </element>
-<element name="R13" library="resistors" package="R-0207/10" value="100K(TH)" x="18.5" y="25" smashed="yes" rot="R90">
-<attribute name="MOUSER" value="71-RN55D-F-100K" x="162.5" y="-63.75" size="1.778" layer="27" rot="R90" display="off"/>
+<element name="R13" library="resistors" package="R-0207/10" value="33K(TH)" x="18.5" y="25" smashed="yes" rot="R90">
 <attribute name="NAME" x="18.5" y="25" size="0.8128" layer="25" ratio="15" rot="R90" align="center"/>
 </element>
-<element name="R15" library="resistors" package="R-0207/10" value="100K(TH)" x="27" y="29" smashed="yes" rot="R180">
-<attribute name="MOUSER" value="71-RN55D-F-100K" x="140.25" y="175.25" size="1.778" layer="27" rot="R180" display="off"/>
+<element name="R15" library="resistors" package="R-0207/10" value="33K(TH)" x="27" y="29" smashed="yes" rot="R180">
 <attribute name="NAME" x="27" y="29" size="0.8128" layer="25" ratio="15" rot="R180" align="center"/>
 </element>

Commit message: M202d Resistor Value Update
Parts:
- R33: value 300K(TH) -> 330K(TH)
Changed lines of the file:
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@@
 <element name="R26" library="resistors" package="R-0207/10" value="15K(TH)" x="14.5" y="25" rot="R90"/>
 <element name="R25" library="resistors" package="R-0207/10" value="470K(TH)" x="27" y="32.5" rot="R180"/>
-<element name="R33" library="resistors" package="R-0207/10" value="300K(TH)" x="12" y="40" rot="R90"/>
+<element name="R33" library="resistors" package="R-0207/10" value="330K(TH)" x="12" y="40" rot="R90"/>
 <element name="R32" library="resistors" package="R-0207/10" value="1K(TH)" x="15" y="32.5" rot="R180">
 <attribute name="MOUSER" value="71-RN55D-F-1.0K" x="22" y="37.5" size="1.778" layer="27" rot="R180" display="off"/>
