File: a111-fader.sch (EAGLE design)
At the start: 50 parts, among them U1 FADER-KNOB-8MM(BLACK/WHITE), U10 NUT-M2-SELFLOCK, U11 FX2-20S-1.27DS, U12 ERM1-5MM, U2 SCREW-M2X8, U3 SCREW-M2X8, U4 NUT-M2-SELFLOCK, U5 NUT-M2-SELFLOCK, U6 FX2-20P-1.27DS, U7 SCREW-M2X8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

Commit message: A111 New VU Indicator preliminary
Parts:
- removed DA2: LM2903N, ic-fairchild:LM2903N
- removed R13: 22K(TH), resistors:22K(TH)
- removed R14: 4K7(TH), resistors:4K7(TH)
- removed R15: 100R(TH), resistors:100R(TH)
- removed R16: 10K(TH), resistors:10K(TH)
- removed R17: 2K2(TH), resistors:2K2(TH)
- removed R18: 1K8(TH), resistors:1K8(TH)
- added DA3: TL072IP, ic-ti:TL072IP
- added R19: 10K(TH), resistors:10K(TH)
- added R20, R21: 100K(TH), resistors:100K(TH)
- added R22: 15K(TH), resistors:15K(TH)
- added R23: 470K(TH), resistors:470K(TH)
- added R24: 300K(TH), resistors:300K(TH)
- added R25, R26: 1K(TH), resistors:1K(TH)
- HL1: value RED/BLUE(2MMX5MM,CC) -> RED/GREEN(2MMX5MM,CC); device optoelectronics:RED/BLUE(2MMX5MM,CC) -> optoelectronics:RED/GREEN(2MMX5MM,CC)
- R6, R8: value 10M(TH) -> 1M(TH); device resistors:10M(TH) -> resistors:1M(TH)
- R7, R9: value 100K(TH) -> 33K(TH); device resistors:100K(TH) -> resistors:33K(TH)
Connections:
- removed net N$26: DA2.1.IN-, R14.1, R15.2
- removed net N$27: DA2.2.IN-, R13.1, R14.2
- removed net N$28: DA2.1.OUT, HL1.A2, R18.1, VT1.C
- removed net N$45: C1.+, C3.2, C7.2, DA1*.V+, DA2*.V+, L1.2
- removed net N$47: C2.-, C4.1, C8.1, DA1*.V-, DA2*.V-, L2.2
- removed net N$48: DA2.2.OUT, HL1.A1, R16.2, R17.1
- removed net N$49: R16.1, VT1.B
- new net N$13: DA3.2.IN-, R19.2, R20.1
- new net N$17: DA3.2.OUT, R20.2, R26.1
- new net N$29: HL1.A2, R26.2, VT1.C
- new net N$30: DA3.1.IN-, R21.1, R22.2, R23.2
- new net N$31: DA3.1.OUT, R21.2, R24.1, R25.1
- new net N$32: R24.2, VT1.B
- new net N$33: HL1.A1, R25.2
- net +15V: now also C1.+, C3.2, C7.2, DA1*.V+, DA3*.V+, L1.2, R23.1; no longer R13.2
- net -15V: now also C2.-, C4.1, C8.1, DA1*.V-, DA3*.V-, L2.2; no longer HL1.K, VT1.E
- net GND: now also HL1.K, R19.1, R22.1, VT1.E; no longer R15.1, R17.2, R18.2
- net N$24: now also DA3.1.IN+, DA3.2.IN+; no longer DA2.1.IN+, DA2.2.IN+
Other:
- moved on the sheet: HL1, U12, VT1

Commit message: A111a Routing
Parts:
- removed R24: 300K(TH), resistors:300K(TH)
- removed R25: 1K(TH), resistors:1K(TH)
- added R13: 10K(TH), resistors:10K(TH)
- added R16: 100K(TH), resistors:100K(TH)
- R19: value 10K(TH) -> 1K(TH); device resistors:10K(TH) -> resistors:1K(TH)
- R20: value 100K(TH) -> 300K(TH); device resistors:100K(TH) -> resistors:300K(TH)
- renumbered DA3 to DA2, R21 to R17, R22 to R15, R23 to R14, R26 to R18
Connections:
- net GND: now also R13.1; no longer R19.1
- net N$13: now also R13.2, R16.1; no longer R19.2, R20.1
- net N$17: now also R16.2; no longer R20.2
- net N$31: now also R19.1, R20.1; no longer R24.1, R25.1
- net N$32: now also R20.2; no longer R24.2
- net N$33: now also R19.2; no longer R25.2
Other:
- moved on the sheet: R19, R20

Commit message: A111a: Resistor Value Update
Parts:
- R20: value 300K(TH) -> 330K(TH); device resistors:300K(TH) -> resistors:330K(TH)
Changed lines of the file:
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@@
 <part name="R15" library="resistors" deviceset="?" device="15K(TH)"/>
 <part name="R14" library="resistors" deviceset="?" device="470K(TH)"/>
-<part name="R20" library="resistors" deviceset="?" device="300K(TH)"/>
+<part name="R20" library="resistors" deviceset="?" device="330K(TH)" value="330K(TH)"/>
 <part name="R19" library="resistors" deviceset="?" device="1K(TH)"/>
 <part name="R18" library="resistors" deviceset="?" device="1K(TH)"/>
