File: d725-pwm-dco.brd (EAGLE design)
At the start: 100 x 50 mm, 62 parts, among them U1 SCREW-M2X8, U10 FX2-20S-1.27DS, U11 ERM1-5MM, U2 SCREW-M2X8, U3 NUT-M2-SELFLOCK, U4 NUT-M2-SELFLOCK, U5 FX2-20P-1.27DS, U6 SCREW-M2X8, U7 SCREW-M2X8, U8 NUT-M2-SELFLOCK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

Commit message: D725 LED Color Change
Parts:
- HL1: value RED/GREEN(2MMX5MM,CC) -> RED/BLUE(2MMX5MM,CC)
Changed lines of the file:
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@@
 <attribute name="MOUSER" value="71-RN55D-F-100/R" x="-30" y="53" size="1.778" layer="27" rot="R270" display="off"/>
 </element>
-<element name="HL1" library="optoelectronics" package="LED2X5-3PIN" value="RED/GREEN(2MMX5MM,CC)" x="9" y="42" rot="R270"/>
+<element name="HL1" library="optoelectronics" package="LED2X5-3PIN" value="RED/BLUE(2MMX5MM,CC)" x="9" y="42" rot="R270"/>
 <element name="U11" library="hardware" package="EMPTY" value="ERM1-5MM" x="2" y="-109"/>
 <element name="O5" library="hardware" package="EMPTY" value="450-AA150(15MM,D,BLACK)" x="60" y="-106">
