File: c122-adsr.brd (EAGLE design)
At the start: 100 x 74 mm, 84 parts, among them U1 SCREW-M2X8, U10 FX2-20S-1.27DS, U11 ERM1-5MM, U12 ERM1-5MM, U2 SCREW-M2X8, U3 NUT-M2-SELFLOCK, U4 NUT-M2-SELFLOCK, U5 FX2-20P-1.27DS, U6 SCREW-M2X8, U7 SCREW-M2X8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

Commit message: C122a LED Color Change
Parts:
- HL1: value RED/GREEN(2MMX5MM,CC) -> RED/BLUE(2MMX5MM,CC)
Changed lines of the file:
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@@
 <attribute name="MOUSER" value="71-RN55D-F-100/R" x="-141" y="70" size="1.778" layer="27" rot="R270" display="off"/>
 </element>
-<element name="HL1" library="optoelectronics" package="LED2X5-3PIN" value="RED/GREEN(2MMX5MM,CC)" x="9" y="66" rot="R90"/>
+<element name="HL1" library="optoelectronics" package="LED2X5-3PIN" value="RED/BLUE(2MMX5MM,CC)" x="9" y="66" rot="R90"/>
 <element name="R1" library="resistors" package="R-0207/10" value="100K(TH)" x="14" y="5">
 <attribute name="MOUSER" value="71-RN55D-F-100K" x="-16" y="-159" size="1.778" layer="27" display="off"/>
