File: m219-bluetooth-input.brd (EAGLE design)
At the start: 100 x 50 mm, 68 parts, among them U1 SCREW-M2X8, U10 FX2-20S-1.27DS, U2 SCREW-M2X8, U3 NUT-M2-SELFLOCK, U4 NUT-M2-SELFLOCK, U5 FX2-20P-1.27DS, U6 SCREW-M2X8, U7 SCREW-M2X8, U8 NUT-M2-SELFLOCK, U9 NUT-M2-SELFLOCK

Commit message: M219 LED Color Update
Parts:
- HL1: value WHITE(2MMX5MM) -> BLUE(2MMX5MM)
- HL2: value ORANGE(2MMX5MM) -> RED(2MMX5MM)
Changed lines of the file:
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@@
 <attribute name="MOUSER" value="660-RK73H2ATTD1001F" x="13" y="37" size="1.778" layer="27" rot="R270" display="off"/>
 </element>
-<element name="HL2" library="optoelectronics" package="LED2X5" value="ORANGE(2MMX5MM)" x="12" y="43" rot="R270"/>
-<element name="HL1" library="optoelectronics" package="LED2X5" value="WHITE(2MMX5MM)" x="9" y="43" rot="R270"/>
+<element name="HL2" library="optoelectronics" package="LED2X5" value="RED(2MMX5MM)" x="12" y="43" rot="R270"/>
+<element name="HL1" library="optoelectronics" package="LED2X5" value="BLUE(2MMX5MM)" x="9" y="43" rot="R270"/>
 <element name="C12" library="capacitors" package="C-0805" value="100N" x="20.5" y="8" rot="R90">
 <attribute name="MOUSER" value="77-VJ0805V104MXBPBC" x="20.5" y="8" size="1.778" layer="27" rot="R90" display="off"/>

Commit message: M219a Routing
Parts:
- HL1: value BLUE(2MMX5MM) -> GREEN(2MMX5MM)
- HL2: value RED(2MMX5MM) -> YELLOW(2MMX5MM)
- moved L1 2.50 mm to (35.0, 41.5), turned to 180 degrees
- moved C11 2.37 mm to (25.0, 31.8), turned to 90 degrees
Routing:
- net +3.3V: track 0.00 -> 65.5 mm, vias 0 -> 2
- net +15V: track 26.7 -> 82.0 mm, vias 1 -> 3
- net N$16: track 0.00 -> 48.9 mm
- net -15V: track 27.7 -> 74.9 mm, vias 2 -> 4
- net N$34: track 0.00 -> 39.1 mm, vias 0 -> 1
- net N$22: track 0.00 -> 35.4 mm
- net N$20: track 0.00 -> 33.1 mm
- net N$30: track 0.00 -> 32.9 mm, vias 0 -> 2
- net N$31: track 0.00 -> 31.4 mm, vias 0 -> 2
- net N$8: track 0.00 -> 30.9 mm
- net N$6: track 0.00 -> 28.1 mm, vias 0 -> 2
- net N$36: track 5.50 -> 23.0 mm
- net N$7: track 5.50 -> 22.0 mm
- net N$29: track 0.00 -> 13.3 mm
- net GND: track 144.1 -> 133.2 mm, vias 7 -> 8
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